Commit message: Added missing frames for sensors and cameras

File: atlas2_description/urdf/atlas2_macro.urdf.xacro (robot description, xacro)
@@ -2,4 +2,7 @@
 <robot xmlns:xacro="http://www.ros.org/wiki/xacro">
     <xacro:include filename="$(find atlas2_description)/urdf/atlas2_model_macro.urdf.xacro" />
+    <xacro:include filename="$(find pointgrey_camera_description)/urdf/pointgrey_flea3.urdf.xacro" />
+    <xacro:include filename="$(find sick_ldmrs_description)/urdf/sick_ldmrs_macros.urdf.xacro" />
+    <xacro:include filename="$(find lms1xx)/urdf/sick_lms1xx.urdf.xacro" />
     <xacro:macro name="atlas2" params="prefix">
         <!-- links -->
@@ -25,4 +28,39 @@
             <child link="${prefix}moving_axis" />
         </joint>
+        <!-- frontal camera -->
+        <xacro:pointgrey_flea3 name="${prefix}front_camera" frame="${prefix}front_camera" />
+        <joint name="${prefix}car_center_to_${prefix}front_camera" type="fixed">
+            <origin xyz="0 0 0.85" rpy="0 0 ${-pi/2}" />
+            <parent link="${prefix}car_center" />
+            <child link="${prefix}front_camera" />
+        </joint>
+        <!-- top camera -->
+        <xacro:pointgrey_flea3 name="${prefix}top_camera" frame="${prefix}top_camera" />
+        <joint name="${prefix}car_center_to_${prefix}top_camera" type="fixed">
+            <origin xyz="0 1.50 1.65" rpy="0 0.4 ${-pi/2}" />
+            <parent link="${prefix}car_center" />
+            <child link="${prefix}top_camera" />
+        </joint>
+        <!-- laser sensor lms_ldmrs400001 -->
+        <xacro:sick_ldmrs name="${prefix}front_laser" />
+        <joint name="${prefix}car_center_to_${prefix}front_laser_mount_link" type="fixed">
+            <origin xyz="0 0 0.4" rpy="0 0 -${pi/2}" />
+            <parent link="${prefix}car_center" />
+            <child link="${prefix}front_laser_mount_link" />
+        </joint>
+        <!-- left lms151 laser -->
+        <xacro:sick_lms1xx frame="${prefix}left_laser" />
+        <joint name="${prefix}car_center_to_${prefix}left_laser" type="fixed">
+            <origin xyz="-0.70 0.05 0.50" rpy="0 0 ${-2.2}" />
+            <parent link="${prefix}car_center" />
+            <child link="${prefix}left_laser" />
+        </joint>
+        <!-- right lms151 laser -->
+        <xacro:sick_lms1xx frame="${prefix}right_laser" />
+        <joint name="${prefix}car_center_to_${prefix}right_laser" type="fixed">
+            <origin xyz="0.70 0.05 0.50" rpy="0 0 ${-1}" />
+            <parent link="${prefix}car_center" />
+            <child link="${prefix}right_laser" />
+        </joint>
     </xacro:macro>
 </robot>

File: atlas2_description/urdf/atlas2_model_macro.urdf.xacro (robot description, xacro)
@@ -4,5 +4,5 @@
         <link name="${prefix}model">
             <visual>
-                <origin xyz="-1.0 0 -0.5" rpy="0 0 0" />
+                <origin xyz="-0.9 0 0" rpy="0 0 0" />
                 <geometry>
                     <mesh filename="package://atlas2_description/meshes/mitsubishi_miev.dae" />

Commit message: sensors elements added

File: atlas2_description/urdf/atlas2_macro.urdf.xacro (robot description, xacro)
@@ -35,4 +35,8 @@
             <child link="${prefix}front_camera" />
         </joint>
+         <sensor name="${prefix}front_camera" update_rate="20">
+             <parent link="${prefix}front_camera"/>
+             <origin xyz="0 0 0" rpy="0 0 0"/>
+         </sensor>
         <!-- top camera -->
         <xacro:pointgrey_flea3 name="${prefix}top_camera" frame="${prefix}top_camera" />
@@ -42,4 +46,8 @@
             <child link="${prefix}top_camera" />
         </joint>
+         <sensor name="${prefix}top_camera" update_rate="20">
+             <parent link="${prefix}top_camera"/>
+             <origin xyz="0 0 0" rpy="0 0 0"/>
+         </sensor>
         <!-- laser sensor lms_ldmrs400001 -->
         <xacro:sick_ldmrs name="${prefix}front_laser" />
@@ -49,4 +57,8 @@
             <child link="${prefix}front_laser_mount_link" />
         </joint>
+         <sensor name="${prefix}front_laser" update_rate="20">
+             <parent link="${prefix}front_laser"/>
+             <origin xyz="0 0 0" rpy="0 0 0"/>
+         </sensor>
         <!-- left lms151 laser -->
         <xacro:sick_lms1xx frame="${prefix}left_laser" />
@@ -56,4 +68,8 @@
             <child link="${prefix}left_laser" />
         </joint>
+         <sensor name="${prefix}left_laser" update_rate="20">
+             <parent link="${prefix}left_laser"/>
+             <origin xyz="0 0 0" rpy="0 0 0"/>
+         </sensor>
         <!-- right lms151 laser -->
         <xacro:sick_lms1xx frame="${prefix}right_laser" />
@@ -63,4 +79,8 @@
             <child link="${prefix}right_laser" />
         </joint>
+         <sensor name="${prefix}right_laser" update_rate="20">
+             <parent link="${prefix}right_laser"/>
+             <origin xyz="0 0 0" rpy="0 0 0"/>
+         </sensor>
     </xacro:macro>
 </robot>

Commit message: Installation explained on readme Source of the car and sensors models is their own packages

File: atlas2_description/urdf/atlas2_macro.urdf.xacro (robot description, xacro)
@@ -35,6 +35,6 @@
             <child link="${prefix}front_camera" />
         </joint>
-         <sensor name="${prefix}front_camera" update_rate="20">
-             <parent link="${prefix}front_camera"/>
+         <sensor name="${prefix}front_camera_optical" update_rate="20">
+             <parent link="${prefix}front_camera_optical"/>
              <origin xyz="0 0 0" rpy="0 0 0"/>
          </sensor>
@@ -46,6 +46,6 @@
             <child link="${prefix}top_camera" />
         </joint>
-         <sensor name="${prefix}top_camera" update_rate="20">
-             <parent link="${prefix}top_camera"/>
+         <sensor name="${prefix}top_camera_optical" update_rate="20">
+             <parent link="${prefix}top_camera_optical"/>
              <origin xyz="0 0 0" rpy="0 0 0"/>
          </sensor>

Commit message: #14 reading calibration_parent and calibration_child elements.

File: atlas2_description/urdf/atlas2_macro.urdf.xacro (robot description, xacro)
@@ -35,7 +35,9 @@
             <child link="${prefix}front_camera" />
         </joint>
-         <sensor name="${prefix}front_camera_optical" update_rate="20">
-             <parent link="${prefix}front_camera_optical"/>
+         <sensor name="${prefix}front_camera" update_rate="20">
+             <parent link="${prefix}front_camera"/>
              <origin xyz="0 0 0" rpy="0 0 0"/>
+             <calibration_parent link="${prefix}car_center"/>
+             <calibration_child link="${prefix}front_camera"/>
          </sensor>
         <!-- top camera -->
@@ -46,7 +48,9 @@
             <child link="${prefix}top_camera" />
         </joint>
-         <sensor name="${prefix}top_camera_optical" update_rate="20">
+         <sensor name="${prefix}top_camera" update_rate="20">
              <parent link="${prefix}top_camera_optical"/>
              <origin xyz="0 0 0" rpy="0 0 0"/>
+             <calibration_parent link="${prefix}car_center"/>
+             <calibration_child link="${prefix}top_camera"/>
          </sensor>
         <!-- laser sensor lms_ldmrs400001 -->
@@ -60,4 +64,6 @@
              <parent link="${prefix}front_laser"/>
              <origin xyz="0 0 0" rpy="0 0 0"/>
+             <calibration_parent link="${prefix}car_center"/>
+             <calibration_child link="${prefix}front_laser_mount_link"/>
          </sensor>
         <!-- left lms151 laser -->
@@ -71,4 +77,6 @@
              <parent link="${prefix}left_laser"/>
              <origin xyz="0 0 0" rpy="0 0 0"/>
+             <calibration_parent link="${prefix}car_center"/>
+             <calibration_child link="${prefix}left_laser"/>
          </sensor>
         <!-- right lms151 laser -->
@@ -82,4 +90,6 @@
              <parent link="${prefix}right_laser"/>
              <origin xyz="0 0 0" rpy="0 0 0"/>
+             <calibration_parent link="${prefix}car_center"/>
+             <calibration_child link="${prefix}right_laser"/>
          </sensor>
     </xacro:macro>

Commit message: camera setup & integration on launch files

File: atlas2_description/urdf/atlas2_macro.urdf.xacro (robot description, xacro)
@@ -29,15 +29,15 @@
         </joint>
         <!-- frontal camera -->
-        <xacro:pointgrey_flea3 name="${prefix}front_camera" frame="${prefix}front_camera" />
-        <joint name="${prefix}car_center_to_${prefix}front_camera" type="fixed">
+        <xacro:pointgrey_flea3 name="${prefix}frontal_camera" frame="${prefix}frontal_camera" />
+        <joint name="${prefix}car_center_to_${prefix}frontal_camera" type="fixed">
             <origin xyz="0 0 0.85" rpy="0 0 ${-pi/2}" />
             <parent link="${prefix}car_center" />
-            <child link="${prefix}front_camera" />
+            <child link="${prefix}frontal_camera" />
         </joint>
-         <sensor name="${prefix}front_camera" update_rate="20">
-             <parent link="${prefix}front_camera"/>
+         <sensor name="${prefix}frontal_camera" update_rate="20">
+             <parent link="${prefix}frontal_camera"/>
              <origin xyz="0 0 0" rpy="0 0 0"/>
              <calibration_parent link="${prefix}car_center"/>
-             <calibration_child link="${prefix}front_camera"/>
+             <calibration_child link="${prefix}frontal_camera"/>
          </sensor>
         <!-- top camera -->

Commit message: #20 created launch file for atlascar2. It is working.

File: atlas2_description/urdf/atlas2_macro.urdf.xacro (robot description, xacro)
@@ -35,10 +35,4 @@
             <child link="${prefix}frontal_camera" />
         </joint>
-         <sensor name="${prefix}frontal_camera" update_rate="20">
-             <parent link="${prefix}frontal_camera"/>
-             <origin xyz="0 0 0" rpy="0 0 0"/>
-             <calibration_parent link="${prefix}car_center"/>
-             <calibration_child link="${prefix}frontal_camera"/>
-         </sensor>
         <!-- top camera -->
         <xacro:pointgrey_flea3 name="${prefix}top_camera" frame="${prefix}top_camera" />
@@ -48,10 +42,4 @@
             <child link="${prefix}top_camera" />
         </joint>
-         <sensor name="${prefix}top_camera" update_rate="20">
-             <parent link="${prefix}top_camera_optical"/>
-             <origin xyz="0 0 0" rpy="0 0 0"/>
-             <calibration_parent link="${prefix}car_center"/>
-             <calibration_child link="${prefix}top_camera"/>
-         </sensor>
         <!-- laser sensor lms_ldmrs400001 -->
         <xacro:sick_ldmrs name="${prefix}front_laser" />
@@ -61,10 +49,4 @@
             <child link="${prefix}front_laser_mount_link" />
         </joint>
-         <sensor name="${prefix}front_laser" update_rate="20">
-             <parent link="${prefix}front_laser"/>
-             <origin xyz="0 0 0" rpy="0 0 0"/>
-             <calibration_parent link="${prefix}car_center"/>
-             <calibration_child link="${prefix}front_laser_mount_link"/>
-         </sensor>
         <!-- left lms151 laser -->
         <xacro:sick_lms1xx frame="${prefix}left_laser" />
@@ -74,10 +56,4 @@
             <child link="${prefix}left_laser" />
         </joint>
-         <sensor name="${prefix}left_laser" update_rate="20">
-             <parent link="${prefix}left_laser"/>
-             <origin xyz="0 0 0" rpy="0 0 0"/>
-             <calibration_parent link="${prefix}car_center"/>
-             <calibration_child link="${prefix}left_laser"/>
-         </sensor>
         <!-- right lms151 laser -->
         <xacro:sick_lms1xx frame="${prefix}right_laser" />
@@ -87,10 +63,4 @@
             <child link="${prefix}right_laser" />
         </joint>
-         <sensor name="${prefix}right_laser" update_rate="20">
-             <parent link="${prefix}right_laser"/>
-             <origin xyz="0 0 0" rpy="0 0 0"/>
-             <calibration_parent link="${prefix}car_center"/>
-             <calibration_child link="${prefix}right_laser"/>
-         </sensor>
     </xacro:macro>
 </robot>

Commit message: #11 renaming also front_laser_mount_link

File: atlas2_description/urdf/atlas2_macro.urdf.xacro (robot description, xacro)
@@ -44,8 +44,8 @@
         <!-- laser sensor lms_ldmrs400001 -->
         <xacro:sick_ldmrs name="${prefix}ldrms" />
-        <joint name="${prefix}car_center_to_${prefix}front_laser_mount_link" type="fixed">
+        <joint name="${prefix}car_center_to_${prefix}ldrms_mount_link" type="fixed">
             <origin xyz="0 0 0.4" rpy="0 0 -${pi/2}" />
             <parent link="${prefix}car_center" />
-            <child link="${prefix}front_laser_mount_link" />
+            <child link="${prefix}ldrms_mount_link" />
         </joint>
         <!-- left lms151 laser -->

Commit message: Readme in construction... almoste ended

File: atlas2_description/urdf/atlas2_macro.urdf.xacro (robot description, xacro)
@@ -3,5 +3,5 @@
     <xacro:include filename="$(find atlas2_description)/urdf/atlas2_model_macro.urdf.xacro" />
     <xacro:include filename="$(find pointgrey_camera_description)/urdf/pointgrey_flea3.urdf.xacro" />
-    <xacro:include filename="$(find sick_ldmrs_description)/urdf/sick_ldmrs_macros.urdf.xacro" />
+    <!--<xacro:include filename="$(find sick_ldmrs_description)/urdf/sick_ldmrs_macros.urdf.xacro" />-->
     <xacro:include filename="$(find lms1xx)/urdf/sick_lms1xx.urdf.xacro" />
     <xacro:macro name="atlas2" params="prefix">
@@ -54,17 +54,17 @@
              <calibration_child link="${prefix}top_camera"/>
          </sensor>
-        <!-- laser sensor lms_ldmrs400001 -->
-        <xacro:sick_ldmrs name="${prefix}front_laser" />
-        <joint name="${prefix}car_center_to_${prefix}front_laser_mount_link" type="fixed">
-            <origin xyz="0 0 0.4" rpy="0 0 -${pi/2}" />
-            <parent link="${prefix}car_center" />
-            <child link="${prefix}front_laser_mount_link" />
-        </joint>
-         <sensor name="${prefix}front_laser" update_rate="20">
-             <parent link="${prefix}front_laser"/>
-             <origin xyz="0 0 0" rpy="0 0 0"/>
-             <calibration_parent link="${prefix}car_center"/>
-             <calibration_child link="${prefix}front_laser_mount_link"/>
-         </sensor>
+        <!--&lt;!&ndash; laser sensor lms_ldmrs400001 &ndash;&gt;-->
+        <!--<xacro:sick_ldmrs name="${prefix}front_laser" />-->
+        <!--<joint name="${prefix}car_center_to_${prefix}front_laser_mount_link" type="fixed">-->
+            <!--<origin xyz="0 0 0.4" rpy="0 0 -${pi/2}" />-->
+            <!--<parent link="${prefix}car_center" />-->
+            <!--<child link="${prefix}front_laser_mount_link" />-->
+        <!--</joint>-->
+         <!--<sensor name="${prefix}front_laser" update_rate="20">-->
+             <!--<parent link="${prefix}front_laser"/>-->
+             <!--<origin xyz="0 0 0" rpy="0 0 0"/>-->
+             <!--<calibration_parent link="${prefix}car_center"/>-->
+             <!--<calibration_child link="${prefix}front_laser_mount_link"/>-->
+         <!--</sensor>-->
         <!-- left lms151 laser -->
         <xacro:sick_lms1xx frame="${prefix}left_laser" />

Commit message: #14 changing names of top cameras

File: atlas2_description/urdf/atlas2_macro.urdf.xacro (robot description, xacro)
@@ -36,16 +36,16 @@
         </joint>
         <!-- top camera -->
-        <xacro:pointgrey_flea3 name="${prefix}top_camera" frame="${prefix}top_camera" />
-        <joint name="${prefix}car_center_to_${prefix}top_camera" type="fixed">
+        <xacro:pointgrey_flea3 name="${prefix}top_right_camera" frame="${prefix}top_right_camera" />
+        <joint name="${prefix}car_center_to_${prefix}top_right_camera" type="fixed">
             <origin xyz="0 1.50 1.65" rpy="0 0.4 ${-pi/2}" />
             <parent link="${prefix}car_center" />
-            <child link="${prefix}top_camera" />
+            <child link="${prefix}top_right_camera" />
         </joint>
         <!-- laser sensor lms_ldmrs400001 -->
-        <xacro:sick_ldmrs name="${prefix}ldrms" />
-        <joint name="${prefix}car_center_to_${prefix}ldrms_mount_link" type="fixed">
+        <xacro:sick_ldmrs name="${prefix}frontal_laser" />
+        <joint name="${prefix}car_center_to_${prefix}frontal_laser_mount_link" type="fixed">
             <origin xyz="0 0 0.4" rpy="0 0 -${pi/2}" />
             <parent link="${prefix}car_center" />
-            <child link="${prefix}ldrms_mount_link" />
+            <child link="${prefix}frontal_laser_mount_link" />
         </joint>
         <!-- left lms151 laser -->

Commit message: Changing xacro

File: atlas2_description/urdf/atlas2_macro.urdf.xacro (robot description, xacro)
@@ -50,17 +50,17 @@
         </joint>
         <!-- left lms151 laser -->
+        <xacro:sick_lms1xx frame="${prefix}right_laser" />
+        <joint name="${prefix}car_center_to_${prefix}right_laser" type="fixed">
+            <origin xyz="-0.70 0.05 0.50" rpy="0 0 ${-2.2}" />
+            <parent link="${prefix}car_center" />
+            <child link="${prefix}right_laser" />
+        </joint>
+        <!-- right lms151 laser -->
         <xacro:sick_lms1xx frame="${prefix}left_laser" />
         <joint name="${prefix}car_center_to_${prefix}left_laser" type="fixed">
-            <origin xyz="-0.70 0.05 0.50" rpy="0 0 ${-2.2}" />
+            <origin xyz="0.70 0.05 0.50" rpy="0 0 ${-1}" />
             <parent link="${prefix}car_center" />
             <child link="${prefix}left_laser" />
         </joint>
-        <!-- right lms151 laser -->
-        <xacro:sick_lms1xx frame="${prefix}right_laser" />
-        <joint name="${prefix}car_center_to_${prefix}right_laser" type="fixed">
-            <origin xyz="0.70 0.05 0.50" rpy="0 0 ${-1}" />
-            <parent link="${prefix}car_center" />
-            <child link="${prefix}right_laser" />
-        </joint>
     </xacro:macro>
 </robot>

Commit message: Changing xacro

File: atlas2_description/urdf/atlas2_macro.urdf.xacro (robot description, xacro)
@@ -7,58 +7,52 @@
     <xacro:macro name="atlas2" params="prefix">
         <!-- links -->
+        <link name="${prefix}base_link" />
         <link name="${prefix}ground" />
-        <link name="${prefix}car_center" />
-        <link name="${prefix}moving_axis" />
         <!-- car model -->
         <xacro:atlas2_model prefix="${prefix}" />
-        <joint name="${prefix}ground_to_${prefix}model" type="fixed">
-            <origin xyz="0 0 0" rpy="0 0 0" />
-            <parent link="${prefix}ground" />
+        <joint name="${prefix}base_link_to_${prefix}model" type="fixed">
+            <origin xyz="0 0 -0.4" rpy="0 0 ${pi/2}" />
+            <parent link="${prefix}base_link" />
             <child link="${prefix}model" />
         </joint>
         <!-- joints -->
-        <joint name="${prefix}ground_to_${prefix}car_center" type="fixed">
-            <origin xyz="0 0 0" rpy="0 0 0" />
-            <parent link="${prefix}ground" />
-            <child link="${prefix}car_center" />
+        <joint name="${prefix}base_link_to_${prefix}ground" type="fixed">
+            <origin xyz="0 0 -0.4" rpy="0 0 0" />
+            <parent link="${prefix}base_link" />
+            <child link="${prefix}ground" />
         </joint>
-        <joint name="${prefix}car_center_to_${prefix}moving_axis" type="fixed">
-            <origin xyz="0 0 0" rpy="0 0 0" />
-            <parent link="${prefix}car_center" />
-            <child link="${prefix}moving_axis" />
+        <!-- top-right-camera -->
+        <xacro:pointgrey_flea3 name="${prefix}top_right_camera" frame="${prefix}top_right_camera" />
+        <joint name="${prefix}base_link_to_${prefix}top_right_camera" type="fixed">
+            <origin xyz="-1.50 -0.12 1.25" rpy="0 0.4 0" />
+            <parent link="${prefix}base_link" />
+            <child link="${prefix}top_right_camera" />
         </joint>
-        <!-- frontal camera -->
-        <xacro:pointgrey_flea3 name="${prefix}frontal_camera" frame="${prefix}frontal_camera" />
-        <joint name="${prefix}car_center_to_${prefix}frontal_camera" type="fixed">
-            <origin xyz="0 0 0.85" rpy="0 0 ${-pi/2}" />
-            <parent link="${prefix}car_center" />
-            <child link="${prefix}frontal_camera" />
-        </joint>
-        <!-- top camera -->
-        <xacro:pointgrey_flea3 name="${prefix}top_right_camera" frame="${prefix}top_right_camera" />
-        <joint name="${prefix}car_center_to_${prefix}top_right_camera" type="fixed">
-            <origin xyz="0 1.50 1.65" rpy="0 0.4 ${-pi/2}" />
-            <parent link="${prefix}car_center" />
-            <child link="${prefix}top_right_camera" />
+        <!-- top-left-camera -->
+        <xacro:pointgrey_flea3 name="${prefix}top_left_camera" frame="${prefix}top_left_camera" />
+        <joint name="${prefix}base_link_to_${prefix}top_left_camera" type="fixed">
+            <origin xyz="-1.50 0.12 1.25" rpy="0 0.4 0" />
+            <parent link="${prefix}base_link" />
+            <child link="${prefix}top_left_camera" />
         </joint>
         <!-- laser sensor lms_ldmrs400001 -->
         <xacro:sick_ldmrs name="${prefix}frontal_laser" />
-        <joint name="${prefix}car_center_to_${prefix}frontal_laser_mount_link" type="fixed">
-            <origin xyz="0 0 0.4" rpy="0 0 -${pi/2}" />
-            <parent link="${prefix}car_center" />
+        <joint name="${prefix}base_link_to_${prefix}frontal_laser_mount_link" type="fixed">
+            <origin xyz="0 0 0" rpy="0 0 0" />
+            <parent link="${prefix}base_link" />
             <child link="${prefix}frontal_laser_mount_link" />
         </joint>
         <!-- left lms151 laser -->
         <xacro:sick_lms1xx frame="${prefix}right_laser" />
-        <joint name="${prefix}car_center_to_${prefix}right_laser" type="fixed">
-            <origin xyz="-0.70 0.05 0.50" rpy="0 0 ${-2.2}" />
-            <parent link="${prefix}car_center" />
+        <joint name="${prefix}base_link_to_${prefix}right_laser" type="fixed">
+            <origin xyz="-0.05 -0.70 0.10" rpy="0 0 ${-0.63}" />
+            <parent link="${prefix}base_link" />
             <child link="${prefix}right_laser" />
         </joint>
         <!-- right lms151 laser -->
         <xacro:sick_lms1xx frame="${prefix}left_laser" />
-        <joint name="${prefix}car_center_to_${prefix}left_laser" type="fixed">
-            <origin xyz="0.70 0.05 0.50" rpy="0 0 ${-1}" />
-            <parent link="${prefix}car_center" />
+        <joint name="${prefix}base_link_to_${prefix}left_laser" type="fixed">
+            <origin xyz="-0.05 0.70  0.10" rpy="0 0 ${0.57}" />
+            <parent link="${prefix}base_link" />
             <child link="${prefix}left_laser" />
         </joint>
