Commit message: #68 extending the atlas2_descrition file with an rgbd camera description

File: atlas2_description/urdf/atlas2_macro.urdf.xacro (robot description, xacro)
@@ -5,4 +5,5 @@
     <xacro:include filename="$(find sick_ldmrs_description)/urdf/sick_ldmrs_macros.urdf.xacro" />
     <xacro:include filename="$(find lms1xx)/urdf/sick_lms1xx.urdf.xacro" />
+    <xacro:include filename="$(find atlas2_description)/urdf/asus_xtion.urdf.xacro" />
     <xacro:macro name="atlas2" params="prefix">
         <!-- links -->
@@ -57,4 +58,11 @@
             <child link="${prefix}left_laser" />
         </joint>
+        <!-- RGB-D camera -->
+        <xacro:asus_camera_model name="${prefix}frontal_rgbd_camera" />
+        <joint name="${prefix}base_link_to_${prefix}frontal_rgbd_camera" type="fixed">
+            <origin xyz="0 0.0  0.20" rpy="0 0 0" />
+            <parent link="${prefix}base_link" />
+            <child link="${prefix}frontal_rgbd_camera_link" />
+        </joint>
     </xacro:macro>
 </robot>

Commit message: #76 done with help from pycharm, should be working but could not confirm ...

File: atlas2_description/urdf/atlas2_macro.urdf.xacro (robot description, xacro)
@@ -59,9 +59,9 @@
         </joint>
         <!-- RGB-D camera -->
-        <xacro:asus_camera_model name="${prefix}frontal_rgbd_camera" />
-        <joint name="${prefix}base_link_to_${prefix}frontal_rgbd_camera" type="fixed">
+        <xacro:asus_camera_model name="${prefix}top_center_rgbd_camera" />
+        <joint name="${prefix}base_link_to_${prefix}top_center_rgbd_camera" type="fixed">
             <origin xyz="0 0.0  0.20" rpy="0 0 0" />
             <parent link="${prefix}base_link" />
-            <child link="${prefix}frontal_rgbd_camera_link" />
+            <child link="${prefix}top_center_rgbd_camera_link" />
         </joint>
     </xacro:macro>

Commit message: https://github.com/lardemua/AtlasCarCalibration/#77

File: atlas2_description/urdf/atlas2_macro.urdf.xacro (robot description, xacro)
@@ -9,5 +9,5 @@
         <!-- links -->
         <link name="${prefix}base_link" />
-        <link name="${prefix}ground" />
+        <link name="${prefix}base_footprint" />
         <!-- car model -->
         <xacro:atlas2_model prefix="${prefix}" />
@@ -19,5 +19,5 @@
         <!-- joints -->
         <joint name="${prefix}base_link_to_${prefix}ground" type="fixed">
-            <origin xyz="0 0 -0.4" rpy="0 0 0" />
+            <origin xyz="0 0 -0.305" rpy="0 0 0" />
             <parent link="${prefix}base_link" />
             <child link="${prefix}ground" />
@@ -26,5 +26,5 @@
         <xacro:pointgrey_flea3 name="${prefix}top_right_camera" frame="${prefix}top_right_camera" />
         <joint name="${prefix}base_link_to_${prefix}top_right_camera" type="fixed">
-            <origin xyz="-1.50 -0.12 1.25" rpy="0 0.4 0" />
+            <origin xyz="-1.55 -0.22 1.35" rpy="0 0.4 0" />
             <parent link="${prefix}base_link" />
             <child link="${prefix}top_right_camera" />
@@ -33,5 +33,5 @@
         <xacro:pointgrey_flea3 name="${prefix}top_left_camera" frame="${prefix}top_left_camera" />
         <joint name="${prefix}base_link_to_${prefix}top_left_camera" type="fixed">
-            <origin xyz="-1.50 0.12 1.25" rpy="0 0.4 0" />
+            <origin xyz="-1.55 0.22 1.35" rpy="0 0.4 0" />
             <parent link="${prefix}base_link" />
             <child link="${prefix}top_left_camera" />
@@ -47,5 +47,5 @@
         <xacro:sick_lms1xx frame="${prefix}right_laser" />
         <joint name="${prefix}base_link_to_${prefix}right_laser" type="fixed">
-            <origin xyz="-0.05 -0.70 0.10" rpy="0 0 ${-0.63}" />
+            <origin xyz="-0.07 -0.76 0.27" rpy="0 0 ${-0.7854}" />
             <parent link="${prefix}base_link" />
             <child link="${prefix}right_laser" />
@@ -54,5 +54,5 @@
         <xacro:sick_lms1xx frame="${prefix}left_laser" />
         <joint name="${prefix}base_link_to_${prefix}left_laser" type="fixed">
-            <origin xyz="-0.05 0.70  0.10" rpy="0 0 ${0.57}" />
+            <origin xyz="-0.07 0.76  0.27" rpy="0 0 ${0.7854}" />
             <parent link="${prefix}base_link" />
             <child link="${prefix}left_laser" />
@@ -61,5 +61,5 @@
         <xacro:asus_camera_model name="${prefix}top_center_rgbd_camera" />
         <joint name="${prefix}base_link_to_${prefix}top_center_rgbd_camera" type="fixed">
-            <origin xyz="0 0.0  0.20" rpy="0 0 0" />
+            <origin xyz="-1.51 0.1 1.27" rpy="0 0.4 0" />
             <parent link="${prefix}base_link" />
             <child link="${prefix}top_center_rgbd_camera_link" />

Commit message: https://github.com/lardemua/AtlasCarCalibration/issues/77

File: atlas2_description/urdf/atlas2_macro.urdf.xacro (robot description, xacro)
@@ -18,8 +18,8 @@
         </joint>
         <!-- joints -->
-        <joint name="${prefix}base_link_to_${prefix}ground" type="fixed">
+        <joint name="${prefix}base_link_to_${prefix}base_footprint" type="fixed">
             <origin xyz="0 0 -0.305" rpy="0 0 0" />
             <parent link="${prefix}base_link" />
-            <child link="${prefix}ground" />
+            <child link="${prefix}base_footprint" />
         </joint>
         <!-- top-right-camera -->
@@ -61,5 +61,5 @@
         <xacro:asus_camera_model name="${prefix}top_center_rgbd_camera" />
         <joint name="${prefix}base_link_to_${prefix}top_center_rgbd_camera" type="fixed">
-            <origin xyz="-1.51 0.1 1.27" rpy="0 0.4 0" />
+            <origin xyz="-1.51 -0.01 1.27" rpy="0 0.4 0" />
             <parent link="${prefix}base_link" />
             <child link="${prefix}top_center_rgbd_camera_link" />

Commit message: #77 placing model_link with parent base_footprint

File: atlas2_description/urdf/atlas2_macro.urdf.xacro (robot description, xacro)
@@ -12,9 +12,4 @@
         <!-- car model -->
         <xacro:atlas2_model prefix="${prefix}" />
-        <joint name="${prefix}base_link_to_${prefix}model" type="fixed">
-            <origin xyz="0 0 -0.4" rpy="0 0 ${pi/2}" />
-            <parent link="${prefix}base_link" />
-            <child link="${prefix}model" />
-        </joint>
         <!-- joints -->
         <joint name="${prefix}base_link_to_${prefix}base_footprint" type="fixed">
@@ -22,4 +17,9 @@
             <parent link="${prefix}base_link" />
             <child link="${prefix}base_footprint" />
+        </joint>
+        <joint name="${prefix}base_footprint_to_${prefix}model" type="fixed">
+            <origin xyz="0 0 0" rpy="0 0 ${pi/2}" />
+            <parent link="${prefix}base_footprint" />
+            <child link="${prefix}model" />
         </joint>
         <!-- top-right-camera -->

Commit message: Creating links and joints in the agrob xacro ...

File: atlas2_description/urdf/atlas2_macro.urdf.xacro (robot description, xacro)
@@ -1,70 +1,70 @@
 <?xml version="1.0"?>
 <robot xmlns:xacro="http://www.ros.org/wiki/xacro">
-    <xacro:include filename="$(find atlas2_description)/urdf/atlas2_model_macro.urdf.xacro" />
-    <xacro:include filename="$(find pointgrey_camera_description)/urdf/pointgrey_flea3.urdf.xacro" />
-    <xacro:include filename="$(find sick_ldmrs_description)/urdf/sick_ldmrs_macros.urdf.xacro" />
-    <xacro:include filename="$(find lms1xx)/urdf/sick_lms1xx.urdf.xacro" />
-    <xacro:include filename="$(find atlas2_description)/urdf/asus_xtion.urdf.xacro" />
-    <xacro:macro name="atlas2" params="prefix">
-        <!-- links -->
-        <link name="${prefix}base_link" />
-        <link name="${prefix}base_footprint" />
-        <!-- car model -->
-        <xacro:atlas2_model prefix="${prefix}" />
-        <!-- joints -->
-        <joint name="${prefix}base_link_to_${prefix}base_footprint" type="fixed">
-            <origin xyz="0 0 -0.305" rpy="0 0 0" />
-            <parent link="${prefix}base_link" />
-            <child link="${prefix}base_footprint" />
-        </joint>
-        <joint name="${prefix}base_footprint_to_${prefix}model" type="fixed">
-            <origin xyz="0 0 0" rpy="0 0 ${pi/2}" />
-            <parent link="${prefix}base_footprint" />
-            <child link="${prefix}model" />
-        </joint>
-        <!-- top-right-camera -->
-        <xacro:pointgrey_flea3 name="${prefix}top_right_camera" frame="${prefix}top_right_camera" />
-        <joint name="${prefix}base_link_to_${prefix}top_right_camera" type="fixed">
-            <origin xyz="-1.55 -0.22 1.35" rpy="0 0.4 0" />
-            <parent link="${prefix}base_link" />
-            <child link="${prefix}top_right_camera" />
-        </joint>
-        <!-- top-left-camera -->
-        <xacro:pointgrey_flea3 name="${prefix}top_left_camera" frame="${prefix}top_left_camera" />
-        <joint name="${prefix}base_link_to_${prefix}top_left_camera" type="fixed">
-            <origin xyz="-1.55 0.22 1.35" rpy="0 0.4 0" />
-            <parent link="${prefix}base_link" />
-            <child link="${prefix}top_left_camera" />
-        </joint>
-        <!-- laser sensor lms_ldmrs400001 -->
-        <xacro:sick_ldmrs name="${prefix}frontal_laser" />
-        <joint name="${prefix}base_link_to_${prefix}frontal_laser_mount_link" type="fixed">
-            <origin xyz="0 0 0" rpy="0 0 0" />
-            <parent link="${prefix}base_link" />
-            <child link="${prefix}frontal_laser_mount_link" />
-        </joint>
-        <!-- left lms151 laser -->
-        <xacro:sick_lms1xx frame="${prefix}right_laser" />
-        <joint name="${prefix}base_link_to_${prefix}right_laser" type="fixed">
-            <origin xyz="-0.07 -0.76 0.27" rpy="0 0 ${-0.7854}" />
-            <parent link="${prefix}base_link" />
-            <child link="${prefix}right_laser" />
-        </joint>
-        <!-- right lms151 laser -->
-        <xacro:sick_lms1xx frame="${prefix}left_laser" />
-        <joint name="${prefix}base_link_to_${prefix}left_laser" type="fixed">
-            <origin xyz="-0.07 0.76  0.27" rpy="0 0 ${0.7854}" />
-            <parent link="${prefix}base_link" />
-            <child link="${prefix}left_laser" />
-        </joint>
-        <!-- RGB-D camera -->
-        <xacro:asus_camera_model name="${prefix}top_center_rgbd_camera" />
-        <joint name="${prefix}base_link_to_${prefix}top_center_rgbd_camera" type="fixed">
-<!--            <origin xyz="-1.510 -0.010 1.397" rpy="-0.000 0.223 -0.000" />-->
-                <origin xyz="-1.510 -0.010 1.338" rpy="-0.000 0.207 -0.000" />
-<!--            <origin xyz="-1.51 -0.01 1.27" rpy="0 0.4 0" />-->
-            <parent link="${prefix}base_link" />
-            <child link="${prefix}top_center_rgbd_camera_link" />
-        </joint>
-    </xacro:macro>
+  <xacro:include filename="$(find atlas2_description)/urdf/atlas2_model_macro.urdf.xacro"/>
+  <xacro:include filename="$(find pointgrey_camera_description)/urdf/pointgrey_flea3.urdf.xacro"/>
+  <xacro:include filename="$(find sick_ldmrs_description)/urdf/sick_ldmrs_macros.urdf.xacro"/>
+  <xacro:include filename="$(find lms1xx)/urdf/sick_lms1xx.urdf.xacro"/>
+  <xacro:include filename="$(find atlas2_description)/urdf/asus_xtion.urdf.xacro"/>
+  <xacro:macro name="atlas2" params="prefix">
+    <!-- links -->
+    <link name="${prefix}base_link"/>
+    <link name="${prefix}base_footprint"/>
+    <!-- car model -->
+    <xacro:atlas2_model prefix="${prefix}"/>
+    <!-- joints -->
+    <joint name="${prefix}base_link_to_${prefix}base_footprint" type="fixed">
+      <origin xyz="0 0 -0.305" rpy="0 0 0"/>
+      <parent link="${prefix}base_link"/>
+      <child link="${prefix}base_footprint"/>
+    </joint>
+    <joint name="${prefix}base_footprint_to_${prefix}model" type="fixed">
+      <origin xyz="0 0 0" rpy="0 0 ${pi/2}"/>
+      <parent link="${prefix}base_footprint"/>
+      <child link="${prefix}model"/>
+    </joint>
+    <!-- top-right-camera -->
+    <xacro:pointgrey_flea3 name="${prefix}top_right_camera" frame="${prefix}top_right_camera"/>
+    <joint name="${prefix}base_link_to_${prefix}top_right_camera" type="fixed">
+      <origin xyz="-1.55 -0.22 1.35" rpy="0 0.4 0"/>
+      <parent link="${prefix}base_link"/>
+      <child link="${prefix}top_right_camera"/>
+    </joint>
+    <!-- top-left-camera -->
+    <xacro:pointgrey_flea3 name="${prefix}top_left_camera" frame="${prefix}top_left_camera"/>
+    <joint name="${prefix}base_link_to_${prefix}top_left_camera" type="fixed">
+      <origin xyz="-1.55 0.22 1.35" rpy="0 0.4 0"/>
+      <parent link="${prefix}base_link"/>
+      <child link="${prefix}top_left_camera"/>
+    </joint>
+    <!-- laser sensor lms_ldmrs400001 -->
+    <xacro:sick_ldmrs name="${prefix}frontal_laser"/>
+    <joint name="${prefix}base_link_to_${prefix}frontal_laser_mount_link" type="fixed">
+      <origin xyz="0 0 0" rpy="0 0 0"/>
+      <parent link="${prefix}base_link"/>
+      <child link="${prefix}frontal_laser_mount_link"/>
+    </joint>
+    <!-- left lms151 laser -->
+    <xacro:sick_lms1xx frame="${prefix}right_laser"/>
+    <joint name="${prefix}base_link_to_${prefix}right_laser" type="fixed">
+      <origin xyz="-0.07 -0.76 0.27" rpy="0 0 ${-0.7854}"/>
+      <parent link="${prefix}base_link"/>
+      <child link="${prefix}right_laser"/>
+    </joint>
+    <!-- right lms151 laser -->
+    <xacro:sick_lms1xx frame="${prefix}left_laser"/>
+    <joint name="${prefix}base_link_to_${prefix}left_laser" type="fixed">
+      <origin xyz="-0.07 0.76  0.27" rpy="0 0 ${0.7854}"/>
+      <parent link="${prefix}base_link"/>
+      <child link="${prefix}left_laser"/>
+    </joint>
+    <!-- RGB-D camera -->
+    <xacro:asus_camera_model name="${prefix}top_center_rgbd_camera"/>
+    <joint name="${prefix}base_link_to_${prefix}top_center_rgbd_camera" type="fixed">
+      <!--            <origin xyz="-1.510 -0.010 1.397" rpy="-0.000 0.223 -0.000" />-->
+      <origin xyz="-1.510 -0.010 1.338" rpy="-0.000 0.207 -0.000"/>
+      <!--            <origin xyz="-1.51 -0.01 1.27" rpy="0 0.4 0" />-->
+      <parent link="${prefix}base_link"/>
+      <child link="${prefix}top_center_rgbd_camera_link"/>
+    </joint>
+  </xacro:macro>
 </robot>
