Commit message: Huge commit, adjusting atlas-core repo to proper naming conventions. Repo now is called atlascar2

File: atlascar2_description/urdf/asus_xtion.urdf.xacro (robot description, xacro)
@@ -22,5 +22,5 @@
           <origin xyz="0 0 0" rpy="0 0 0" />
           <geometry>
-            <mesh filename="package://atlas2_description/meshes/asus_xtion/asus_xtion_simple.dae"/>
+            <mesh filename="package://atlascar2_description/meshes/asus_xtion/asus_xtion_simple.dae"/>
           </geometry>
         </visual>
@@ -36,5 +36,5 @@
           <origin xyz="0 0 0" rpy="0 0 0" />
           <geometry>
-            <mesh filename="package://atlas2_description/meshes/asus_xtion/asus_xtion_simple.dae"/>
+            <mesh filename="package://atlascar2_description/meshes/asus_xtion/asus_xtion_simple.dae"/>
           </geometry>
         </collision>

File: atlascar2_description/urdf/atlascar2_macro.urdf.xacro (robot description, xacro)
@@ -1,15 +1,15 @@
 <?xml version="1.0"?>
 <robot xmlns:xacro="http://www.ros.org/wiki/xacro">
-  <xacro:include filename="$(find atlas2_description)/urdf/atlas2_model_macro.urdf.xacro"/>
+  <xacro:include filename="$(find atlascar2_description)/urdf/atlascar2_model_macro.urdf.xacro"/>
   <xacro:include filename="$(find pointgrey_camera_description)/urdf/pointgrey_flea3.urdf.xacro"/>
   <xacro:include filename="$(find sick_ldmrs_description)/urdf/sick_ldmrs_macros.urdf.xacro"/>
   <xacro:include filename="$(find lms1xx)/urdf/sick_lms1xx.urdf.xacro"/>
-  <xacro:include filename="$(find atlas2_description)/urdf/asus_xtion.urdf.xacro"/>
-  <xacro:macro name="atlas2" params="prefix">
+  <xacro:include filename="$(find atlascar2_description)/urdf/asus_xtion.urdf.xacro"/>
+  <xacro:macro name="atlascar2" params="prefix">
     <!-- links -->
     <link name="${prefix}base_link"/>
     <link name="${prefix}base_footprint"/>
     <!-- car model -->
-    <xacro:atlas2_model prefix="${prefix}"/>
+    <xacro:atlascar2_model prefix="${prefix}"/>
     <!-- joints -->
     <joint name="${prefix}base_link_to_${prefix}base_footprint" type="fixed">

File: atlascar2_description/urdf/atlascar2_model_macro.urdf.xacro (robot description, xacro)
@@ -1,10 +1,10 @@
 <?xml version="1.0"?>
 <robot xmlns:xacro="http://www.ros.org/wiki/xacro">
-    <xacro:macro name="atlas2_model" params="prefix">
+    <xacro:macro name="atlascar2_model" params="prefix">
         <link name="${prefix}model">
             <visual>
                 <origin xyz="-0.9 0 0" rpy="0 0 0" />
                 <geometry>
-                    <mesh filename="package://atlas2_description/meshes/mitsubishi_miev.dae" />
+                    <mesh filename="package://atlascar2_description/meshes/mitsubishi_miev.dae" />
                 </geometry>
             </visual>

File: atlascar2_description/urdf/atlascar2_posopt_macro.urdf.xacro (robot description, xacro)
@@ -1,15 +1,15 @@
 <?xml version="1.0"?>
 <robot xmlns:xacro="http://www.ros.org/wiki/xacro">
-    <xacro:include filename="$(find atlas2_description)/urdf/atlas2_model_macro.urdf.xacro" />
+    <xacro:include filename="$(find atlascar2_description)/urdf/atlascar2_model_macro.urdf.xacro" />
     <xacro:include filename="$(find pointgrey_camera_description)/urdf/pointgrey_flea3.urdf.xacro" />
     <xacro:include filename="$(find sick_ldmrs_description)/urdf/sick_ldmrs_macros.urdf.xacro" />
     <xacro:include filename="$(find lms1xx)/urdf/sick_lms1xx.urdf.xacro" />
-    <xacro:include filename="$(find atlas2_description)/urdf/asus_xtion.urdf.xacro" />
-    <xacro:macro name="atlas2" params="prefix">
+    <xacro:include filename="$(find atlascar2_description)/urdf/asus_xtion.urdf.xacro" />
+    <xacro:macro name="atlascar2" params="prefix">
         <!-- links -->
         <link name="${prefix}base_link" />
         <link name="${prefix}base_footprint" />
         <!-- car model -->
-        <xacro:atlas2_model prefix="${prefix}" />
+        <xacro:atlascar2_model prefix="${prefix}" />
         <!-- joints -->
         <joint name="${prefix}base_link_to_${prefix}base_footprint" type="fixed">
