Commit message: damping added

File: atlascar2_description/urdf/wheel.urdf.xacro (robot description, xacro)
@@ -5,4 +5,6 @@
   <xacro:property name="steer_effort"   value="10.0"/>
   <xacro:property name="steer_velocity" value="5.0"/>
+  <xacro:property name="inertia" value="0.5"/>
+  <xacro:property name="damping" value="0.5"/>
   <xacro:macro name="front_steer" params="name parent radius thickness length width axel_offset steer_height *origin">
     <link name="${name}_steer_link">
@@ -10,5 +12,5 @@
         <origin xyz="0 0 0" rpy="0 0 0"/>
         <mass value="1"/>
-        <inertia ixx="1" ixy="0" ixz="0" iyy="1" iyz="0" izz="1"/>
+        <inertia ixx="${inertia}" ixy="0" ixz="0" iyy="${inertia}" iyz="0" izz="${inertia}"/>
       </inertial>
       <visual>
@@ -33,4 +35,5 @@
              lower="${-180.0 * deg_to_rad}" upper="${180.0 * deg_to_rad}"
              velocity="${steer_velocity}"/>
+      <dynamics damping="${damping}" friction="0.0"/>
      </joint>
            <!-- Transmission is important to link the joints and the controller -->
@@ -40,4 +43,5 @@
       <joint name="${name}_steer_joint">
         <hardwareInterface>hardware_interface/PositionJointInterface</hardwareInterface>
+        <dynamics damping="${damping}" friction="0.0"/>
       </joint>
       <mechanicalReduction>1</mechanicalReduction>
@@ -53,5 +57,5 @@
         <origin xyz="0 0 0" rpy="0 0 0"/>
         <mass value="1"/>
-        <inertia ixx="1" ixy="0" ixz="0" iyy="1" iyz="0" izz="1"/>
+        <inertia ixx="${inertia}" ixy="0" ixz="0" iyy="${inertia}" iyz="0" izz="${inertia}"/>
       </inertial>
       <visual>
@@ -74,4 +78,5 @@
       <!--xacro:insert_block name="origin"/-->
       <axis xyz="0 0 1"/>
+      <dynamics damping="${damping}" friction="0.0"/>
       <limit effort="${steer_effort}"
              lower="${-180.0 * deg_to_rad}" upper="${180.0 * deg_to_rad}"
@@ -82,5 +87,5 @@
         <origin xyz="0 0 0" rpy="0 0 0"/>
         <mass value="1"/>
-        <inertia ixx="10" ixy="0" ixz="0" iyy="10" iyz="0" izz="10"/>
+        <inertia ixx="${inertia}" ixy="0" ixz="0" iyy="${inertia}" iyz="0" izz="${inertia}"/>
       </inertial>
       <visual>
@@ -102,4 +107,5 @@
       <origin xyz="0 0 ${-steer_height}" rpy="${-90 * deg_to_rad} 0 0"/>
       <axis xyz="0 0 1"/>
+      <dynamics damping="${damping}" friction="0.0"/>
     </joint>
     <!-- Transmission is important to link the joints and the controller -->
@@ -109,4 +115,5 @@
       <joint name="${name}_steer_joint">
         <hardwareInterface>hardware_interface/EffortJointInterface</hardwareInterface>
+        <dynamics damping="${damping}" friction="0.0"/>
       </joint>
       <mechanicalReduction>1</mechanicalReduction>
@@ -118,4 +125,5 @@
       <joint name="${name}_wheel_joint">
         <hardwareInterface>hardware_interface/EffortJointInterface</hardwareInterface>
+        <dynamics damping="${damping}" friction="0.0"/>
       </joint>
       <mechanicalReduction>1</mechanicalReduction>
@@ -134,5 +142,5 @@
         <origin xyz="0 0 0" rpy="0 0 0"/>
         <mass value="1"/>
-        <inertia ixx="1" ixy="0" ixz="0" iyy="1" iyz="0" izz="1"/>
+        <inertia ixx="${inertia}" ixy="0" ixz="0" iyy="${inertia}" iyz="0" izz="${inertia}"/>
       </inertial>
       <visual>
@@ -154,4 +162,5 @@
       <xacro:insert_block name="origin"/>
       <axis xyz="0 0 1"/>
+      <dynamics damping="${damping}" friction="0.0"/>
     </joint>
     <!-- Transmission is important to link the joints and the controller -->
@@ -160,5 +169,6 @@
       <actuator name="${name}_wheel_joint_motor"/>
       <joint name="${name}_wheel_joint">
-              <hardwareInterface>hardware_interface/VelocityJointInterface</hardwareInterface>
+          <hardwareInterface>hardware_interface/VelocityJointInterface</hardwareInterface>
+          <dynamics damping="${damping}" friction="0.0"/>
       </joint>
       <mechanicalReduction>1</mechanicalReduction>
@@ -174,5 +184,5 @@
         <origin xyz="0 0 0" rpy="0 0 0"/>
         <mass value="1"/>
-        <inertia ixx="1" ixy="0" ixz="0" iyy="1" iyz="0" izz="1"/>
+        <inertia ixx="${inertia}" ixy="0" ixz="0" iyy="${inertia}" iyz="0" izz="${inertia}"/>
       </inertial>
       <visual>
@@ -194,4 +204,5 @@
       <xacro:insert_block name="origin"/>
       <axis xyz="0 0 1"/>
+      <dynamics damping="${damping}" friction="0.0"/>
     </joint>
     <!-- Transmission is important to link the joints and the controller -->
@@ -200,5 +211,6 @@
       <actuator name="${name}_wheel_joint_motor"/>
       <joint name="${name}_wheel_joint">
-              <hardwareInterface>hardware_interface/EffortJointInterface</hardwareInterface>
+          <hardwareInterface>hardware_interface/EffortJointInterface</hardwareInterface>
+          <dynamics damping="${damping}" friction="0.0"/>
       </joint>
       <mechanicalReduction>1</mechanicalReduction>

Commit message: front steer joint looks like it dows nothing

File: atlascar2_description/urdf/wheel.urdf.xacro (robot description, xacro)
@@ -3,8 +3,8 @@
   <xacro:property name="steer_radius" value="0.05" /> <!-- Link 1 -->
   <xacro:property name="steer_thickness" value="0.02" /> <!-- Link 1 -->
-  <xacro:property name="steer_effort"   value="10.0"/>
+  <xacro:property name="steer_effort"   value="15.0"/>
   <xacro:property name="steer_velocity" value="5.0"/>
-  <xacro:property name="inertia" value="0.5"/>
-  <xacro:property name="damping" value="0.5"/>
+  <xacro:property name="inertia" value="0.05"/>
+  <xacro:property name="damping" value="0.02"/>
   <xacro:macro name="front_steer" params="name parent radius thickness length width axel_offset steer_height *origin">
     <link name="${name}_steer_link">

Commit message: wheels not right

File: atlascar2_description/urdf/wheel.urdf.xacro (robot description, xacro)
@@ -75,9 +75,9 @@
     </link>
     <joint name="${name}_steer_joint" type="revolute">
-<!--      <parent link="${parent}_link"/>-->
-      <parent link="front_steer_link"/>
+      <parent link="${parent}_link"/>
+<!--      <parent link="front_steer_link"/>-->
       <child link="${name}_steer_link"/>
-<!--      <origin xyz="${length/2-axel_offset} ${right_left*(width/2+axel_offset)} ${steer_height}" rpy="0 0 0"/>-->
-      <origin xyz="0 ${right_left*(width/2+axel_offset)} 0" rpy="0 0 0"/>
+      <origin xyz="${length/2-axel_offset} ${right_left*(width/2+axel_offset)} ${steer_height}" rpy="0 0 0"/>
+<!--      <origin xyz="0 ${right_left*(width/2+axel_offset)} 0" rpy="0 0 0"/>-->
       <!--xacro:insert_block name="origin"/-->
       <axis xyz="0 0 1"/>

Commit message: simulation working

File: atlascar2_description/urdf/wheel.urdf.xacro (robot description, xacro)
@@ -6,12 +6,12 @@
   <xacro:property name="steer_velocity" value="5.0"/>
   <xacro:property name="inertia" value="0.002"/>
-  <xacro:property name="inertia_yy" value="0.02"/>
-  <xacro:property name="damping" value="0.02"/>
-  <xacro:property name="friction" value="0.02" />
+  <xacro:property name="inertia_yy" value="0.002"/>
+  <xacro:property name="damping" value="0.0"/>
+  <xacro:property name="friction" value="0.0" />
   <xacro:macro name="front_steer" params="name parent radius thickness length width axel_offset steer_height *origin">
     <link name="${name}_steer_link">
       <inertial>
         <origin xyz="0 0 0" rpy="0 0 0"/>
-        <mass value="1"/>
+        <mass value="0.5"/>
         <inertia ixx="${inertia}" ixy="0" ixz="0" iyy="${inertia_yy}" iyz="0" izz="${inertia}"/>
       </inertial>
@@ -58,5 +58,5 @@
       <inertial>
         <origin xyz="0 0 0" rpy="0 0 0"/>
-        <mass value="1"/>
+        <mass value="0.5"/>
         <inertia ixx="${inertia}" ixy="0" ixz="0" iyy="${inertia_yy}" iyz="0" izz="${inertia}"/>
       </inertial>
@@ -90,5 +90,5 @@
       <inertial>
         <origin xyz="0 0 0" rpy="0 0 0"/>
-        <mass value="1"/>
+        <mass value="0.5"/>
         <inertia ixx="${inertia}" ixy="0" ixz="0" iyy="${inertia_yy}" iyz="0" izz="${inertia}"/>
       </inertial>
@@ -147,5 +147,5 @@
       <inertial>
         <origin xyz="0 0 0" rpy="0 0 0"/>
-        <mass value="1"/>
+        <mass value="0.5"/>
         <inertia ixx="${inertia}" ixy="0" ixz="0" iyy="${inertia_yy}" iyz="0" izz="${inertia}"/>
       </inertial>
