Commit message: changed inertia values

File: atlascar2_description/urdf/atlascar2_ackermann_v2.urdf.xacro (robot description, xacro)
@@ -21,10 +21,12 @@
   <!-- Links: inertial,visual,collision -->
   <link name="base_link">
-<!--    <inertial>-->
-<!--      &lt;!&ndash; origin is relative &ndash;&gt;-->
-<!--      <origin xyz="0 0 0" rpy="0 0 0"/>-->
-<!--      <mass value="5"/>-->
-<!--      <inertia ixx="5" ixy="0" ixz="0" iyy="5" iyz="0" izz="5"/>-->
-<!--    </inertial>-->
+    <inertial>
+      <!-- origin is relative -->
+      <origin xyz="0 0 0" rpy="0 0 0"/>
+      <mass value="5"/>
+      <inertia ixx="5" ixy="0" ixz="0"
+               iyy="5" iyz="0"
+               izz="5"/>
+    </inertial>
     <visual>
       <geometry>
@@ -82,6 +84,8 @@
   </xacro:rear_wheel_lr>
   <gazebo>
-      <plugin name="gazebo_ros_control" filename="libgazebo_ros_control.so"/>
-  </gazebo>
+  <plugin name="gazebo_ros_control" filename="libgazebo_ros_control.so">
+    <robotNamespace>/atlascar2</robotNamespace>
+  </plugin>
+</gazebo>
   <!-- Colour -->
   <gazebo reference="base_link">

File: atlascar2_description/urdf/wheel.urdf.xacro (robot description, xacro)
@@ -10,5 +10,5 @@
         <origin xyz="0 0 0" rpy="0 0 0"/>
         <mass value="1"/>
-        <inertia ixx="0.2" ixy="0" ixz="0" iyy="0.2" iyz="0" izz="0.2"/>
+        <inertia ixx="1" ixy="0" ixz="0" iyy="1" iyz="0" izz="1"/>
       </inertial>
       <visual>
@@ -34,4 +34,14 @@
              velocity="${steer_velocity}"/>
      </joint>
+           <!-- Transmission is important to link the joints and the controller -->
+    <transmission name="${name}_steer_joint_trans">
+      <type>transmission_interface/SimpleTransmission</type>
+      <actuator name="${name}_steer_joint_motor"/>
+      <joint name="${name}_steer_joint">
+        <hardwareInterface>hardware_interface/PositionJointInterface</hardwareInterface>
+      </joint>
+      <mechanicalReduction>1</mechanicalReduction>
+      <motorTorqueConstant>1</motorTorqueConstant>
+    </transmission>
     <gazebo reference="${name}_steer_link">
       <material>Gazebo/Yellow</material>
@@ -43,5 +53,5 @@
         <origin xyz="0 0 0" rpy="0 0 0"/>
         <mass value="1"/>
-        <inertia ixx="0.2" ixy="0" ixz="0" iyy="0.2" iyz="0" izz="0.2"/>
+        <inertia ixx="1" ixy="0" ixz="0" iyy="1" iyz="0" izz="1"/>
       </inertial>
       <visual>
@@ -72,5 +82,5 @@
         <origin xyz="0 0 0" rpy="0 0 0"/>
         <mass value="1"/>
-        <inertia ixx="0.2" ixy="0" ixz="0" iyy="0.2" iyz="0" izz="0.2"/>
+        <inertia ixx="10" ixy="0" ixz="0" iyy="10" iyz="0" izz="10"/>
       </inertial>
       <visual>
@@ -124,5 +134,5 @@
         <origin xyz="0 0 0" rpy="0 0 0"/>
         <mass value="1"/>
-        <inertia ixx="0.2" ixy="0" ixz="0" iyy="0.2" iyz="0" izz="0.2"/>
+        <inertia ixx="1" ixy="0" ixz="0" iyy="1" iyz="0" izz="1"/>
       </inertial>
       <visual>
@@ -150,5 +160,5 @@
       <actuator name="${name}_wheel_joint_motor"/>
       <joint name="${name}_wheel_joint">
-              <hardwareInterface>hardware_interface/EffortJointInterface</hardwareInterface>
+              <hardwareInterface>hardware_interface/VelocityJointInterface</hardwareInterface>
       </joint>
       <mechanicalReduction>1</mechanicalReduction>
@@ -164,5 +174,5 @@
         <origin xyz="0 0 0" rpy="0 0 0"/>
         <mass value="1"/>
-        <inertia ixx="0.2" ixy="0" ixz="0" iyy="0.2" iyz="0" izz="0.2"/>
+        <inertia ixx="1" ixy="0" ixz="0" iyy="1" iyz="0" izz="1"/>
       </inertial>
       <visual>

Commit message: wheels not right

File: atlascar2_description/urdf/atlascar2_ackermann_v2.urdf.xacro (robot description, xacro)
@@ -85,5 +85,4 @@
   <gazebo>
   <plugin name="gazebo_ros_control" filename="libgazebo_ros_control.so">
-    <robotNamespace>/atlascar2</robotNamespace>
   </plugin>
 </gazebo>

File: atlascar2_description/urdf/wheel.urdf.xacro (robot description, xacro)
@@ -5,6 +5,8 @@
   <xacro:property name="steer_effort"   value="15.0"/>
   <xacro:property name="steer_velocity" value="5.0"/>
-  <xacro:property name="inertia" value="0.05"/>
+  <xacro:property name="inertia" value="0.002"/>
+  <xacro:property name="inertia_yy" value="0.02"/>
   <xacro:property name="damping" value="0.02"/>
+  <xacro:property name="friction" value="0.02" />
   <xacro:macro name="front_steer" params="name parent radius thickness length width axel_offset steer_height *origin">
     <link name="${name}_steer_link">
@@ -12,5 +14,5 @@
         <origin xyz="0 0 0" rpy="0 0 0"/>
         <mass value="1"/>
-        <inertia ixx="${inertia}" ixy="0" ixz="0" iyy="${inertia}" iyz="0" izz="${inertia}"/>
+        <inertia ixx="${inertia}" ixy="0" ixz="0" iyy="${inertia_yy}" iyz="0" izz="${inertia}"/>
       </inertial>
       <visual>
@@ -35,5 +37,5 @@
              lower="${-180.0 * deg_to_rad}" upper="${180.0 * deg_to_rad}"
              velocity="${steer_velocity}"/>
-      <dynamics damping="${damping}" friction="0.0"/>
+      <dynamics damping="${damping}" friction="${friction}"/>
      </joint>
            <!-- Transmission is important to link the joints and the controller -->
@@ -57,5 +59,5 @@
         <origin xyz="0 0 0" rpy="0 0 0"/>
         <mass value="1"/>
-        <inertia ixx="${inertia}" ixy="0" ixz="0" iyy="${inertia}" iyz="0" izz="${inertia}"/>
+        <inertia ixx="${inertia}" ixy="0" ixz="0" iyy="${inertia_yy}" iyz="0" izz="${inertia}"/>
       </inertial>
       <visual>
@@ -73,10 +75,12 @@
     </link>
     <joint name="${name}_steer_joint" type="revolute">
-      <parent link="${parent}_link"/>
+<!--      <parent link="${parent}_link"/>-->
+      <parent link="front_steer_link"/>
       <child link="${name}_steer_link"/>
-      <origin xyz="${length/2-axel_offset} ${right_left*(width/2+axel_offset)} ${steer_height}" rpy="0 0 0"/>
+<!--      <origin xyz="${length/2-axel_offset} ${right_left*(width/2+axel_offset)} ${steer_height}" rpy="0 0 0"/>-->
+      <origin xyz="0 ${right_left*(width/2+axel_offset)} 0" rpy="0 0 0"/>
       <!--xacro:insert_block name="origin"/-->
       <axis xyz="0 0 1"/>
-      <dynamics damping="${damping}" friction="0.0"/>
+      <dynamics damping="${damping}" friction="${friction}"/>
       <limit effort="${steer_effort}"
              lower="${-180.0 * deg_to_rad}" upper="${180.0 * deg_to_rad}"
@@ -87,5 +91,5 @@
         <origin xyz="0 0 0" rpy="0 0 0"/>
         <mass value="1"/>
-        <inertia ixx="${inertia}" ixy="0" ixz="0" iyy="${inertia}" iyz="0" izz="${inertia}"/>
+        <inertia ixx="${inertia}" ixy="0" ixz="0" iyy="${inertia_yy}" iyz="0" izz="${inertia}"/>
       </inertial>
       <visual>
@@ -103,9 +107,11 @@
     </link>
     <joint name="${name}_wheel_joint" type="continuous">
+<!--      <parent link="front_steer_link"/>-->
       <parent link="${name}_steer_link"/>
       <child link="${name}_wheel_link"/>
-      <origin xyz="0 0 ${-steer_height}" rpy="${-90 * deg_to_rad} 0 0"/>
-      <axis xyz="0 0 1"/>
-      <dynamics damping="${damping}" friction="0.0"/>
+<!--      <origin xyz="0 ${right_left*(width/2+axel_offset)} ${-steer_height}" rpy="${-90 * deg_to_rad} 0 0"/>-->
+      <origin xyz="0 0 ${-steer_height}" rpy="${-90 * deg_to_rad} 0 0"/>-->
+      <axis xyz="0 0 1"/>
+      <dynamics damping="${damping}" friction="${friction}"/>
     </joint>
     <!-- Transmission is important to link the joints and the controller -->
@@ -114,6 +120,6 @@
       <actuator name="${name}_steer_joint_motor"/>
       <joint name="${name}_steer_joint">
-        <hardwareInterface>hardware_interface/EffortJointInterface</hardwareInterface>
-        <dynamics damping="${damping}" friction="0.0"/>
+        <hardwareInterface>hardware_interface/PositionJointInterface</hardwareInterface>
+        <dynamics damping="${damping}" friction="${friction}"/>
       </joint>
       <mechanicalReduction>1</mechanicalReduction>
@@ -125,5 +131,5 @@
       <joint name="${name}_wheel_joint">
         <hardwareInterface>hardware_interface/EffortJointInterface</hardwareInterface>
-        <dynamics damping="${damping}" friction="0.0"/>
+        <dynamics damping="${damping}" friction="${friction}"/>
       </joint>
       <mechanicalReduction>1</mechanicalReduction>
@@ -142,5 +148,5 @@
         <origin xyz="0 0 0" rpy="0 0 0"/>
         <mass value="1"/>
-        <inertia ixx="${inertia}" ixy="0" ixz="0" iyy="${inertia}" iyz="0" izz="${inertia}"/>
+        <inertia ixx="${inertia}" ixy="0" ixz="0" iyy="${inertia_yy}" iyz="0" izz="${inertia}"/>
       </inertial>
       <visual>
@@ -162,5 +168,5 @@
       <xacro:insert_block name="origin"/>
       <axis xyz="0 0 1"/>
-      <dynamics damping="${damping}" friction="0.0"/>
+      <dynamics damping="${damping}" friction="${friction}"/>
     </joint>
     <!-- Transmission is important to link the joints and the controller -->
@@ -170,5 +176,5 @@
       <joint name="${name}_wheel_joint">
           <hardwareInterface>hardware_interface/VelocityJointInterface</hardwareInterface>
-          <dynamics damping="${damping}" friction="0.0"/>
+          <dynamics damping="${damping}" friction="${friction}"/>
       </joint>
       <mechanicalReduction>1</mechanicalReduction>
@@ -184,5 +190,5 @@
         <origin xyz="0 0 0" rpy="0 0 0"/>
         <mass value="1"/>
-        <inertia ixx="${inertia}" ixy="0" ixz="0" iyy="${inertia}" iyz="0" izz="${inertia}"/>
+        <inertia ixx="${inertia}" ixy="0" ixz="0" iyy="${inertia_yy}" iyz="0" izz="${inertia}"/>
       </inertial>
       <visual>
@@ -204,5 +210,5 @@
       <xacro:insert_block name="origin"/>
       <axis xyz="0 0 1"/>
-      <dynamics damping="${damping}" friction="0.0"/>
+      <dynamics damping="${damping}" friction="${friction}"/>
     </joint>
     <!-- Transmission is important to link the joints and the controller -->
@@ -212,5 +218,5 @@
       <joint name="${name}_wheel_joint">
           <hardwareInterface>hardware_interface/EffortJointInterface</hardwareInterface>
-          <dynamics damping="${damping}" friction="0.0"/>
+          <dynamics damping="${damping}" friction="${friction}"/>
       </joint>
       <mechanicalReduction>1</mechanicalReduction>

Commit message: simulation working

File: atlascar2_description/urdf/atlascar2_ackermann_v2.urdf.xacro (robot description, xacro)
@@ -24,8 +24,8 @@
       <!-- origin is relative -->
       <origin xyz="0 0 0" rpy="0 0 0"/>
-      <mass value="5"/>
-      <inertia ixx="5" ixy="0" ixz="0"
-               iyy="5" iyz="0"
-               izz="5"/>
+      <mass value="2"/>
+      <inertia ixx="2" ixy="0" ixz="0"
+               iyy="2" iyz="0"
+               izz="2"/>
     </inertial>
     <visual>

Commit message: xacro with the atlascar body done and working

File: atlascar2_description/urdf/atlascar2_ackermann_v2.urdf.xacro (robot description, xacro)
@@ -6,11 +6,4 @@
   <xacro:include filename="wheel.urdf.xacro"/>
   <xacro:property name="deg_to_rad" value="0.01745329251994329577"/>
-  <!-- Constants for robot dimensions -->
-<!--  <xacro:property name="length" value="3.475" />-->
-<!--  <xacro:property name="width" value="1.475" />-->
-<!--  <xacro:property name="wheel_radius" value="0.285" /> &lt;!&ndash; Link 1 &ndash;&gt;-->
-<!--  <xacro:property name="thickness" value="0.145" /> &lt;!&ndash; Link 2 &ndash;&gt;-->
-<!--  <xacro:property name="axel_offset" value="1.5" /> &lt;!&ndash; Space btw top of beam and the each joint &ndash;&gt;-->
-<!--  <xacro:property name="steer_offset" value="0.02" /> &lt;!&ndash; Link 1 &ndash;&gt;-->
     <xacro:property name="length" value="0.5" />
   <xacro:property name="width" value="0.3" />
