Commit message: xacro with the atlascar body done and working

File: atlascar2_description/urdf/atlascar2_body_macro.urdf.xacro (robot description, xacro)
@@ -21,8 +21,8 @@
       <!-- origin is relative -->
       <origin xyz="0 0 0" rpy="0 0 0"/>
-      <mass value="1000"/>
-      <inertia ixx="700" ixy="0" ixz="0"
-               iyy="700" iyz="0"
-               izz="700"/>
+      <mass value="2"/>
+      <inertia ixx="1" ixy="0" ixz="0"
+               iyy="1" iyz="0"
+               izz="1"/>
     </inertial>
     <visual>
@@ -84,5 +84,4 @@
   <gazebo>
     <plugin name="gazebo_ros_control" filename="libgazebo_ros_control.so">
-<!--      <robotNamespace>/atlascar2</robotNamespace>-->
       <robotSimType>steer_bot_hardware_gazebo/SteerBotHardwareGazebo</robotSimType>
     </plugin>

File: atlascar2_description/urdf/atlascar2_wheel.urdf.xacro (robot description, xacro)
@@ -5,13 +5,14 @@
   <xacro:property name="steer_effort"   value="15.0"/>
   <xacro:property name="steer_velocity" value="5.0"/>
-  <xacro:property name="inertia" value="30"/>
-  <xacro:property name="inertia_yy" value="30"/>
-  <xacro:property name="damping" value="5.0"/>
-  <xacro:property name="friction" value="5.0" />
+  <xacro:property name="mass" value="0.3"/>
+  <xacro:property name="inertia" value="0.02"/>
+  <xacro:property name="inertia_yy" value="0.002"/>
+  <xacro:property name="damping" value="0"/>
+  <xacro:property name="friction" value="0" />
   <xacro:macro name="front_steer" params="name parent radius thickness length width axel_offset steer_height *origin">
     <link name="${name}_steer_link">
       <inertial>
         <origin xyz="0 0 0" rpy="0 0 0"/>
-        <mass value="100"/>
+        <mass value="${mass}"/>
         <inertia ixx="${inertia}" ixy="0" ixz="0" iyy="${inertia_yy}" iyz="0" izz="${inertia}"/>
       </inertial>
@@ -55,5 +56,5 @@
       <inertial>
         <origin xyz="0 0 0" rpy="0 0 0"/>
-        <mass value="100"/>
+        <mass value="${mass}"/>
         <inertia ixx="${inertia}" ixy="0" ixz="0" iyy="${inertia_yy}" iyz="0" izz="${inertia}"/>
       </inertial>
@@ -85,5 +86,5 @@
       <inertial>
         <origin xyz="0 0 0" rpy="0 0 0"/>
-        <mass value="100"/>
+        <mass value="${mass}"/>
         <inertia ixx="${inertia}" ixy="0" ixz="0" iyy="${inertia_yy}" iyz="0" izz="${inertia}"/>
       </inertial>
@@ -136,9 +137,12 @@
       <inertial>
         <origin xyz="0 0 0" rpy="0 0 0"/>
-        <mass value="100"/>
+        <mass value="${mass}"/>
         <inertia ixx="${inertia}" ixy="0" ixz="0" iyy="${inertia_yy}" iyz="0" izz="${inertia}"/>
       </inertial>
 <!--      <visual>-->
 <!--        <origin xyz="0 0 0" rpy="0 0 0"/>-->
+<!--        <geometry>-->
+<!--          <cylinder radius="${wheel_radius}" length="${thickness}"/>-->
+<!--        </geometry>-->
 <!--      </visual>-->
       <collision>
@@ -153,5 +157,5 @@
       <child link="${name}_wheel_link"/>
       <xacro:insert_block name="origin"/>
-      <axis xyz="0 0 0"/>
+      <axis xyz="1 0 0"/>
       <dynamics damping="${damping}" friction="${friction}"/>
     </joint>
@@ -172,5 +176,5 @@
       <inertial>
         <origin xyz="0 0 0" rpy="0 0 0"/>
-        <mass value="100"/>
+        <mass value="${mass}"/>
         <inertia ixx="${inertia}" ixy="0" ixz="0" iyy="${inertia_yy}" iyz="0" izz="${inertia}"/>
       </inertial>

Commit message: xacro with the atlascar body done and working

File: atlascar2_description/urdf/atlascar2_body_macro.urdf.xacro (robot description, xacro)
@@ -29,5 +29,5 @@
       <origin xyz=" ${length/2} ${-width/2 - 0.15} ${-wheel_radius + 0.05}" rpy="0 0 ${90*deg_to_rad}"/>
       <geometry>
-        <mesh filename="$(find atlascar2_description)/meshes/atlascar2_nowheels.dae"/>
+        <mesh filename="file:///$(find atlascar2_description)/meshes/atlascar2_nowheels.dae"/>
       </geometry>
     </visual>

File: atlascar2_description/urdf/atlascar2_wheel.urdf.xacro (robot description, xacro)
@@ -92,5 +92,5 @@
         <origin xyz="0 0 0" rpy="0 0 0"/>
         <geometry>
-          <mesh filename="$(find atlascar2_description)/meshes/atlascar2_wheel.dae"/>
+          <mesh filename="file:///$(find atlascar2_description)/meshes/atlascar2_wheel.dae"/>
         </geometry>
       </visual>
@@ -182,5 +182,5 @@
         <origin xyz="0 0 0" rpy="0 0 0"/>
         <geometry>
-            <mesh filename="$(find atlascar2_description)/meshes/atlascar2_wheel.dae"/>
+            <mesh filename="file:///$(find atlascar2_description)/meshes/atlascar2_wheel.dae"/>
         </geometry>
       </visual>
