Commit message: #lardemua/atom#366 Fixed meshes.

File: atlascar2_description/urdf/atlascar2_ackermann.urdf.xacro (robot description, xacro)
@@ -42,18 +42,4 @@
     <xacro:property name="chassis_mass" value="2.788"/>
     <!--
-     battery_dist is the distance between the inner edges of the
-           batteries. battery_comp_depth is the battery compartment depth.
-           battery_length is measured along the x axis, battery_width
-           along the y axis, and battery_height along the z axis.
-    -->
-    <xacro:property name="battery_x_offset" value="0.055"/>
-    <xacro:property name="battery_dist" value="0.065"/>
-    <xacro:property name="battery_comp_depth" value="0.02"/>
-    <xacro:property name="battery_comp_angle" value="0.34906585"/>
-    <xacro:property name="battery_length" value="0.8"/>
-    <xacro:property name="battery_width" value="0.047"/>
-    <xacro:property name="battery_height" value="0.024"/>
-    <xacro:property name="battery_mass" value="0.5025"/>
-    <!--
      hub_dia and tire_dia are the diameters of the hub and tire,
            respectively. hex_hub_depth is the distance that the hex hub is
@@ -112,7 +98,4 @@
     <xacro:property name="servo_stall_torque" value="5649"/>
     <xacro:property name="servo_no_load_speed" value="4553"/>
-    <material name="battery_mat">
-        <color rgba="0 0 1 1"/>
-    </material>
     <material name="chassis_mat">
         <color rgba="0.894 0.054 0.027 1"/>
@@ -157,41 +140,4 @@
                      iyz="0" izz="${mass * (inner_rad * inner_rad + outer_rad * outer_rad) / 2}"/>
         </inertial>
-    </xacro:macro>
-    <!-- Battery -->
-    <xacro:macro name="battery" params="prefix reflect">
-        <joint name="chassis_to_${prefix}_battery" type="fixed">
-            <parent link="chassis"/>
-            <child link="${prefix}_battery_offset"/>
-            <origin xyz="${battery_x_offset - battery_length / 2} ${reflect * battery_dist / 2} 0"
-                    rpy="${reflect * battery_comp_angle} 0 0"/>
-        </joint>
-        <link name="${prefix}_battery_offset">
-            <xacro:null_inertial/>
-        </link>
-        <joint name="offset_to_${prefix}_battery" type="fixed">
-            <parent link="${prefix}_battery_offset"/>
-            <child link="${prefix}_battery"/>
-            <origin xyz="0 ${reflect * battery_width / 2} ${(battery_height / 2) - battery_comp_depth}"/>
-        </joint>
-        <link name="${prefix}_battery">
-            <visual>
-                <geometry>
-                    <box size="${battery_length} ${battery_width} ${battery_height}"/>
-                </geometry>
-                <material name="battery_mat"/>
-            </visual>
-            <collision>
-                <geometry>
-                    <box size="${battery_length} ${battery_width} ${battery_height}"/>
-                </geometry>
-            </collision>
-            <xacro:solid_cuboid_inertial width="${battery_length}" depth="${battery_width}" height="${battery_height}"
-                                         mass="${battery_mass}">
-                <origin/>
-            </xacro:solid_cuboid_inertial>
-        </link>
-        <gazebo reference="${prefix}_battery">
-            <material>Gazebo/Blue</material>
-        </gazebo>
     </xacro:macro>
     <!-- Shock absorber -->
@@ -255,6 +201,7 @@
             <visual>
                 <origin xyz="0 ${lr_reflect * (axle_length - (tire_width / 2 - hex_hub_depth))} 0"/>
+                <origin rpy="${degrees_90} 0 0"/>
                 <geometry>
-                    <mesh filename="$(find atlascar2_description)/meshes/atlascar2_wheel.stl"/>
+                    <mesh filename="$(find atlascar2_description)/meshes/atlascar2_wheel.dae"/>
                 </geometry>
                 <material name="tire_mat"/>
@@ -328,5 +275,6 @@
         <visual>
             <!-- <origin xyz="0 0 0"/> -->
-            <origin xyz="-1.7575 -0.91 -0.295" rpy="${degrees_90} 0.02 ${degrees_90}"/>
+<!--            <origin xyz="-1.7575 -0.91 -0.295" rpy="0 0 0"/>-->
+            <origin xyz="0 0 0" rpy="0 0 0"/>
             <geometry>
                 <!--
@@ -355,7 +303,4 @@
         <child link="chassis"/>
     </joint>
-    <!-- Batteries -->
-    <xacro:battery prefix="left" reflect="1"/>
-    <xacro:battery prefix="right" reflect="-1"/>
     <!-- Wheels -->
     <xacro:front_wheel lr_prefix="left" fr_prefix="front" lr_reflect="1" fr_reflect="1"/>

Commit message: #lardemua/atom#366 Car spawn done correctly.

File: atlascar2_description/urdf/atlascar2_ackermann.urdf.xacro (robot description, xacro)
@@ -36,9 +36,12 @@
            along the y axis, and chassis_height along the z axis.
     -->
-    <xacro:property name="chassis_length" value="2.55"/>
-    <!-- c -->
-    <xacro:property name="chassis_width" value="0.7"/>
-    <xacro:property name="chassis_height" value="0.01"/>
-    <xacro:property name="chassis_mass" value="2.788"/>
+<!--    <xacro:property name="chassis_length" value="2.55"/>-->
+<!--    <xacro:property name="chassis_width" value="0.7"/>-->
+<!--    <xacro:property name="chassis_height" value="0.01"/>-->
+<!--    <xacro:property name="chassis_mass" value="2.788"/>-->
+    <xacro:property name="chassis_length" value="3.475"/>
+    <xacro:property name="chassis_width" value="1.475"/>
+    <xacro:property name="chassis_height" value="1.61"/>
+    <xacro:property name="chassis_mass" value="1100"/>
     <!--
      hub_dia and tire_dia are the diameters of the hub and tire,
@@ -51,5 +54,5 @@
     <xacro:property name="tire_dia" value="0.570"/>
     <!-- c -->
-    <xacro:property name="tire_width" value="0.0889"/>
+    <xacro:property name="tire_width" value="0.145"/>
     <xacro:property name="hex_hub_depth" value="0.01445"/>
     <xacro:property name="wheel_mass" value="15.0"/>
@@ -200,6 +203,6 @@
         <link name="${lr_prefix}_${fr_prefix}_wheel">
             <visual>
-                <origin xyz="0 ${lr_reflect * (axle_length - (tire_width / 2 - hex_hub_depth))} 0"/>
-                <origin rpy="${degrees_90} 0 0"/>
+<!--                <origin xyz="0 ${lr_reflect * (axle_length - (tire_width / 2 - hex_hub_depth))} 1" rpy="0 ${-lr_reflect * degrees_90} 0"/>-->
+                <origin xyz="0 0 0" rpy="0 ${-lr_reflect * degrees_90} 0"/>
                 <geometry>
                     <mesh filename="$(find atlascar2_description)/meshes/atlascar2_wheel.dae"/>
@@ -217,5 +220,5 @@
         </link>
         <gazebo reference="${lr_prefix}_${fr_prefix}_wheel">
-            <material>Gazebo/Black</material>
+            <material>Gazebo/Grey</material>
         </gazebo>
     </xacro:macro>
@@ -275,10 +278,6 @@
         <visual>
             <!-- <origin xyz="0 0 0"/> -->
-<!--            <origin xyz="-1.7575 -0.91 -0.295" rpy="0 0 0"/>-->
-            <origin xyz="0 0 0" rpy="0 0 0"/>
+            <origin xyz=" ${chassis_length/2} ${-chassis_width/2 - 0.15} 0" rpy="0 0 ${degrees_90}"/>
             <geometry>
-                <!--
-                 <box size="${chassis_length} ${chassis_width} ${chassis_height}"/>
-                -->
                 <mesh filename="$(find atlascar2_description)/meshes/atlascar2_nowheels.dae"/>
             </geometry>
@@ -286,13 +285,13 @@
         </visual>
         <collision>
-            <origin xyz="0 0 ${-chassis_height / 2}"/>
+            <origin xyz="0 0 ${(chassis_height + tire_dia)/ 2}"/>
             <geometry>
-                <box size="${chassis_length} ${chassis_width} ${chassis_height}"/>
+                <box size="${chassis_length} ${chassis_width} ${chassis_height - tire_dia}"/>
             </geometry>
         </collision>
-        <xacro:solid_cuboid_inertial width="${chassis_length}" depth="${chassis_width}" height="${chassis_height}"
-                                     mass="${chassis_mass}">
-            <origin xyz="0 0 ${-chassis_height / 2}"/>
-        </xacro:solid_cuboid_inertial>
+    <xacro:solid_cuboid_inertial width="${chassis_length}" depth="${chassis_width}" height="${chassis_height - tire_dia}"
+                                 mass="${chassis_mass}">
+        <origin xyz="0 0 ${(chassis_height - tire_dia) / 2}"/>
+    </xacro:solid_cuboid_inertial>
     </link>
     <gazebo reference="chassis">

Commit message: #lardemua/atom#366 Controller running with problems moving straight

File: atlascar2_description/urdf/atlascar2_ackermann.urdf.xacro (robot description, xacro)
@@ -43,5 +43,5 @@
     <xacro:property name="chassis_width" value="1.475"/>
     <xacro:property name="chassis_height" value="1.61"/>
-    <xacro:property name="chassis_mass" value="1100"/>
+    <xacro:property name="chassis_mass" value="11"/>
     <!--
      hub_dia and tire_dia are the diameters of the hub and tire,
@@ -65,5 +65,5 @@
     <xacro:property name="wheelbase" value="2.55"/>
     <!-- c -->
-    <xacro:property name="hex_hub_dist" value="1.310"/>
+    <xacro:property name="hex_hub_dist" value="1.475"/>
     <!-- c -->
     <xacro:property name="axle_length" value="0.03"/>
@@ -157,5 +157,5 @@
             <type>transmission_interface/SimpleTransmission</type>
             <joint name="${lr_prefix}_${fr_prefix}_shock">
-                <hardwareInterface>EffortJointInterface</hardwareInterface>
+                <hardwareInterface>hardware_interface/EffortJointInterface</hardwareInterface>
             </joint>
             <actuator name="${lr_prefix}_${fr_prefix}_shock_act">
@@ -164,5 +164,5 @@
                              with ROS Hydro.
                 -->
-                <hardwareInterface>EffortJointInterface</hardwareInterface>
+                <hardwareInterface>hardware_interface/EffortJointInterface</hardwareInterface>
                 <mechanicalReduction>1</mechanicalReduction>
             </actuator>
@@ -190,5 +190,5 @@
             <type>transmission_interface/SimpleTransmission</type>
             <joint name="${lr_prefix}_${fr_prefix}_axle">
-                <hardwareInterface>EffortJointInterface</hardwareInterface>
+                <hardwareInterface>hardware_interface/EffortJointInterface</hardwareInterface>
             </joint>
             <actuator name="${lr_prefix}_${fr_prefix}_axle_act">
@@ -197,5 +197,5 @@
                              with ROS Hydro.
                 -->
-                <hardwareInterface>EffortJointInterface</hardwareInterface>
+                <hardwareInterface>hardware_interface/EffortJointInterface</hardwareInterface>
                 <mechanicalReduction>1</mechanicalReduction>
             </actuator>
@@ -240,5 +240,5 @@
             <type>transmission_interface/SimpleTransmission</type>
             <joint name="${lr_prefix}_steering_joint">
-                <hardwareInterface>EffortJointInterface</hardwareInterface>
+                <hardwareInterface>hardware_interface/EffortJointInterface</hardwareInterface>
             </joint>
             <actuator name="${lr_prefix}_steering_act">
@@ -247,5 +247,5 @@
                              with ROS Hydro.
                 -->
-                <hardwareInterface>EffortJointInterface</hardwareInterface>
+                <hardwareInterface>hardware_interface/EffortJointInterface</hardwareInterface>
                 <mechanicalReduction>1</mechanicalReduction>
             </actuator>
@@ -277,6 +277,5 @@
     <link name="chassis">
         <visual>
-            <!-- <origin xyz="0 0 0"/> -->
-            <origin xyz=" ${chassis_length/2} ${-chassis_width/2 - 0.15} 0" rpy="0 0 ${degrees_90}"/>
+            <origin xyz=" ${chassis_length/2} ${-chassis_width/2 - 0.15} ${-tire_dia/2 + 0.1}" rpy="0 0 ${degrees_90}"/>
             <geometry>
                 <mesh filename="$(find atlascar2_description)/meshes/atlascar2_nowheels.dae"/>
@@ -284,10 +283,10 @@
             <material name="chassis_mat"/>
         </visual>
-        <collision>
-            <origin xyz="0 0 ${(chassis_height + tire_dia)/ 2}"/>
-            <geometry>
-                <box size="${chassis_length} ${chassis_width} ${chassis_height - tire_dia}"/>
-            </geometry>
-        </collision>
+<!--        <collision>-->
+<!--            <origin xyz="0 0 ${(chassis_height + tire_dia)/ 2}"/>-->
+<!--            <geometry>-->
+<!--                <box size="${chassis_length} ${chassis_width - 0.5} ${chassis_height - 3*tire_dia/2}"/>-->
+<!--            </geometry>-->
+<!--        </collision>-->
     <xacro:solid_cuboid_inertial width="${chassis_length}" depth="${chassis_width}" height="${chassis_height - tire_dia}"
                                  mass="${chassis_mass}">

Commit message: #lardemua/atom#366 Updated urdf

File: atlascar2_description/urdf/atlascar2_ackermann.urdf.xacro (robot description, xacro)
@@ -56,5 +56,5 @@
     <xacro:property name="tire_width" value="0.145"/>
     <xacro:property name="hex_hub_depth" value="0.01445"/>
-    <xacro:property name="wheel_mass" value="15.0"/>
+    <xacro:property name="wheel_mass" value="0.3"/>
     <!--
      hex_hub_dist is the distance between left and right hex hubs when
@@ -208,5 +208,5 @@
                     <mesh filename="$(find atlascar2_description)/meshes/atlascar2_wheel.dae"/>
                 </geometry>
-                <material name="tire_mat"/>
+<!--                <material name="tire_mat"/>-->
             </visual>
             <collision>
@@ -283,10 +283,10 @@
             <material name="chassis_mat"/>
         </visual>
-<!--        <collision>-->
-<!--            <origin xyz="0 0 ${(chassis_height + tire_dia)/ 2}"/>-->
-<!--            <geometry>-->
-<!--                <box size="${chassis_length} ${chassis_width - 0.5} ${chassis_height - 3*tire_dia/2}"/>-->
-<!--            </geometry>-->
-<!--        </collision>-->
+        <collision>
+            <origin xyz="0 0 ${(chassis_height + tire_dia)/ 2}"/>
+            <geometry>
+                <box size="${chassis_length} ${chassis_width} ${chassis_height - 3*tire_dia/2}"/>
+            </geometry>
+        </collision>
     <xacro:solid_cuboid_inertial width="${chassis_length}" depth="${chassis_width}" height="${chassis_height - tire_dia}"
                                  mass="${chassis_mass}">

Commit message: #lardemua/atom#366 Wobbling issue disappeared

File: atlascar2_description/urdf/atlascar2_ackermann.urdf.xacro (robot description, xacro)
@@ -206,4 +206,5 @@
                 <origin xyz="0 0 0" rpy="0 ${-lr_reflect * degrees_90} 0"/>
                 <geometry>
+<!--                    <cylinder radius="${tire_dia / 2}" length="${tire_width}"/>-->
                     <mesh filename="$(find atlascar2_description)/meshes/atlascar2_wheel.dae"/>
                 </geometry>
@@ -211,5 +212,5 @@
             </visual>
             <collision>
-                <origin xyz="0 ${lr_reflect * (axle_length - (tire_width / 2 - hex_hub_depth))} 0"/>
+                <origin xyz="0 0 0"/>
                 <geometry>
                     <cylinder radius="${tire_dia / 2}" length="${tire_width}"/>

Commit message: #lardemua/atom#366 Hard limit for steering hand

File: atlascar2_description/urdf/atlascar2_ackermann.urdf.xacro (robot description, xacro)
@@ -206,8 +206,7 @@
                 <origin xyz="0 0 0" rpy="0 ${-lr_reflect * degrees_90} 0"/>
                 <geometry>
-<!--                    <cylinder radius="${tire_dia / 2}" length="${tire_width}"/>-->
                     <mesh filename="$(find atlascar2_description)/meshes/atlascar2_wheel.dae"/>
                 </geometry>
-<!--                <material name="tire_mat"/>-->
+                <material name="tire_mat"/>
             </visual>
             <collision>

Commit message: #lardemua/atom#366 Small adjustments to the models and adding the tf_preffix atlascar2

File: atlascar2_description/urdf/atlascar2_ackermann.urdf.xacro (robot description, xacro)
@@ -204,5 +204,5 @@
             <visual>
 <!--                <origin xyz="0 ${lr_reflect * (axle_length - (tire_width / 2 - hex_hub_depth))} 1" rpy="0 ${-lr_reflect * degrees_90} 0"/>-->
-                <origin xyz="0 0 0" rpy="0 ${-lr_reflect * degrees_90} 0"/>
+                <origin xyz="0 0 ${lr_reflect * 0.05}" rpy="0 ${-lr_reflect * degrees_90} 0"/>
                 <geometry>
                     <mesh filename="$(find atlascar2_description)/meshes/atlascar2_wheel.dae"/>
@@ -211,5 +211,5 @@
             </visual>
             <collision>
-                <origin xyz="0 0 0"/>
+                <origin xyz="0 0 ${lr_reflect * 0.05}"/>
                 <geometry>
                     <cylinder radius="${tire_dia / 2}" length="${tire_width}"/>

Commit message: #lardemua/atom#366 Small adjustments to the name of files and the colision box of the vehicle

File: atlascar2_description/urdf/atlascar2_ackermann.urdf.xacro (robot description, xacro)
@@ -284,7 +284,8 @@
         </visual>
         <collision>
-            <origin xyz="0 0 ${(chassis_height + tire_dia)/ 2}"/>
+            <origin xyz="0 0 ${(chassis_height)/ 2}"/>
             <geometry>
-                <box size="${chassis_length} ${chassis_width} ${chassis_height - 3*tire_dia/2}"/>
+                <box size="${chassis_length} ${chassis_width - 2 * tire_width} ${chassis_height - tire_dia/2}"/>
+<!--                <box size="${chassis_length} ${chassis_width} ${chassis_height - 3*tire_dia/2}"/>-->
             </geometry>
         </collision>
