Commit message: #32 Added sensors with gazebo bug

File: atlascar2_description/urdf/atlascar2_ackermann_VLP.urdf.xacro (robot description, xacro)
@@ -7,4 +7,7 @@
     <xacro:include filename="$(find pointgrey_camera_description)/urdf/pointgrey_flea3.urdf.xacro"/>
     <xacro:include filename="$(find velodyne_description)/urdf/VLP-16.urdf.xacro"/>
+    <xacro:include filename="$(find pointgrey_camera_description)/urdf/pointgrey_flea3.urdf.xacro"/>
+    <xacro:include filename="$(find sick_ldmrs_description)/urdf/sick_ldmrs_macros.urdf.xacro"/>
+    <xacro:include filename="$(find lms1xx)/urdf/sick_lms1xx.urdf.xacro"/>
     <xacro:property name="deg_to_rad" value="0.01745329251994329577"/>
     <!-- Constants for robot dimensions -->
@@ -86,5 +89,5 @@
     </joint>
     <!-- top velodyne lidar -->
-    <xacro:VLP-16 name="VLP_lidar" parent="base_link" topic="/lidar_1/velodyne_points">
+    <xacro:VLP-16 name="top_lidar" parent="base_link" topic="/top_laser/cloud">
       <origin xyz="0 0 ${1.35+height_offset}" rpy="0 0 0"/>
     </xacro:VLP-16>
@@ -97,4 +100,25 @@
         <origin xyz="${-length/2+axel_offset_x} 0 0" rpy="${-90 * deg_to_rad} 0 ${-90 * deg_to_rad}"/>
     </xacro:rear_wheel>
+    <!-- laser sensor lms_ldmrs400001 -->
+    <xacro:sick_ldmrs name="frontal_laser"/>
+    <joint name="base_link_to_frontal_laser_mount_link" type="fixed">
+      <origin xyz="${length/2 + length_offset} 0 ${height_offset}" rpy="0 0 0"/>
+      <parent link="base_link"/>
+      <child link="frontal_laser_mount_link"/>
+    </joint>
+    <!-- left lms151 laser -->
+    <xacro:sick_lms1xx frame="left_laser" topic="/left_laser/scan"/>
+    <joint name="base_link_to_left_laser" type="fixed">
+      <origin xyz="${length/2 + length_offset - 0.08} 0.76 ${height_offset+0.27}" rpy="0 0 ${0.7854}"/>
+      <parent link="base_link"/>
+      <child link="left_laser"/>
+    </joint>
+    <!-- right lms151 laser -->
+    <xacro:sick_lms1xx frame="right_laser" topic="/right_laser/scan"/>
+    <joint name="base_link_to_right_laser" type="fixed">
+      <origin xyz="${length/2 + length_offset - 0.08} -0.76 ${height_offset+0.27}" rpy="0 0 ${-0.7854}"/>
+      <parent link="base_link"/>
+      <child link="right_laser"/>
+    </joint>
     <!-- Wheels -->
     <xacro:front_wheel_lr name="front_right" parent="base" radius="${wheel_radius}" thickness="${thickness}"

Commit message: #32 trying to remove tf_preffix

File: atlascar2_description/urdf/atlascar2_ackermann_VLP.urdf.xacro (robot description, xacro)
@@ -21,5 +21,4 @@
     <xacro:property name="axel_offset_y" value="0" /> <!-- Space btw top of beam and the each joint -->
     <xacro:property name="steer_offset" value="0.02" /> <!-- Link 1 -->
-    <xacro:property name="vehicle_name" value="atlascar2"/> <!-- Name of vehicle-->
     <!-- Add car macro -->
     <xacro:atlascar2 length="${length}" width="${width}" height="${height}" wheel_radius="${wheel_radius}"/>
