Commit message: #32 New calibration package, with errors

File: atlascar2_calibration/urdf/initial_estimate.urdf.xacro (robot description, xacro)
@@ -1,72 +1,124 @@
 <?xml version="1.0"?>
-<robot xmlns:xacro="http://www.ros.org/wiki/xacro" name="atlas">
-  <xacro:include filename="$(find atlascar2_description)/urdf/atlascar2_model_macro.urdf.xacro"/>
-  <xacro:include filename="$(find pointgrey_camera_description)/urdf/pointgrey_flea3.urdf.xacro"/>
-  <xacro:include filename="$(find sick_ldmrs_description)/urdf/sick_ldmrs_macros.urdf.xacro"/>
-  <xacro:include filename="$(find lms1xx)/urdf/sick_lms1xx.urdf.xacro"/>
-  <xacro:include filename="$(find atlascar2_description)/urdf/asus_xtion.urdf.xacro"/>
-  <xacro:macro name="atlascar2" params="prefix">
-    <!-- links -->
-    <link name="${prefix}base_link"/>
-    <link name="${prefix}base_footprint"/>
-    <!-- car model -->
-    <xacro:atlascar2_model prefix="${prefix}"/>
-    <!-- joints -->
-    <joint name="${prefix}base_link_to_${prefix}base_footprint" type="fixed">
-      <origin xyz="0 0 -0.305" rpy="0 0 0"/>
-      <parent link="${prefix}base_link"/>
-      <child link="${prefix}base_footprint"/>
+<robot name="atlascar2" xmlns:xacro="http://www.ros.org/wiki/xacro">
+    <!--
+    Robot model taken from http://wiki.ros.org/pr2_mechanism/Tutorials/SImple%20URDF-Controller%20Example
+    -->
+    <xacro:include filename="$(find atlascar2_description)/urdf/atlascar2_wheel.urdf.xacro"/>
+    <xacro:include filename="$(find pointgrey_camera_description)/urdf/pointgrey_flea3.urdf.xacro"/>
+    <xacro:include filename="$(find velodyne_description)/urdf/VLP-16.urdf.xacro"/>
+    <xacro:property name="deg_to_rad" value="0.01745329251994329577"/>
+    <!-- Constants for robot dimensions -->
+    <xacro:property name="length" value="3.475" />
+    <xacro:property name="width" value="1.475" />
+    <xacro:property name="height" value="1.61"/>
+    <xacro:property name="length_offset" value="0.2"/>
+    <xacro:property name="height_offset" value="0.1"/>
+    <xacro:property name="wheel_radius" value="0.285" /> <!-- Link 1 -->
+    <xacro:property name="thickness" value="0.145" /> <!-- Link 2 -->
+    <!--  we need two because the car isn't a square-->
+    <xacro:property name="axel_offset_x" value="0.5" /> <!-- Space btw top of beam and the each joint -->
+    <xacro:property name="axel_offset_y" value="0" /> <!-- Space btw top of beam and the each joint -->
+    <xacro:property name="steer_offset" value="0.02" /> <!-- Link 1 -->
+    <!-- Links: inertial,visual,collision -->
+    <link name="base_link">
+        <inertial>
+            <!-- origin is relative -->
+            <origin xyz="0 0 0" rpy="0 0 0"/>
+            <mass value="2"/>
+            <inertia ixx="1" ixy="0" ixz="0"
+                     iyy="1" iyz="0"
+                     izz="1"/>
+        </inertial>
+        <visual>
+            <origin xyz=" ${length/2} ${-width/2 - 0.15} ${-wheel_radius + 0.05}" rpy="0 0 ${90*deg_to_rad}"/>
+            <geometry>
+                <mesh filename="file:///$(find atlascar2_description)/meshes/atlascar2_nowheels.dae"/>
+            </geometry>
+        </visual>
+        <collision>
+            <!-- origin is relative -->
+            <origin xyz=" 0 0 ${-wheel_radius + height/2}"/>
+            <geometry>
+                <box size="${length - 0.1} ${width} ${height/2}"/>
+            </geometry>
+        </collision>
+    </link>
+    <link name="top_collision">
+        <collision>
+            <origin xyz="${-length/7} 0 0"/>
+            <geometry>
+                <box size="${length/2} ${width} ${height/2}"/>
+            </geometry>
+        </collision>
+    </link>
+    <joint name="base_link_to_top_collision" type="fixed">
+        <origin xyz="0 0 ${height/2}" rpy="0 0 0"/>
+        <parent link="base_link"/>
+        <child link="top_collision"/>
     </joint>
-    <joint name="${prefix}base_footprint_to_${prefix}model" type="fixed">
-      <origin xyz="0 0 0" rpy="0 0 ${pi/2}"/>
-      <parent link="${prefix}base_footprint"/>
-      <child link="${prefix}model"/>
+    <link name="base_footprint">
+        <collision>
+            <origin xyz="0 0 0"/>
+            <geometry>
+                <sphere radius="0.00000001"/>
+            </geometry>
+        </collision>
+    </link>
+    <joint name="base_footprint_joint" type="fixed">
+        <origin xyz="0 0 ${wheel_radius}" rpy="0 0 0"/>
+        <child link="base_link"/>
+        <parent link="base_footprint"/>
     </joint>
-    <!-- top-right-camera -->
-    <xacro:pointgrey_flea3 name="${prefix}top_right_camera" frame="${prefix}top_right_camera"/>
-    <joint name="${prefix}base_link_to_${prefix}top_right_camera" type="fixed">
-      <origin xyz="-1.55 -0.22 1.35" rpy="0 0.4 0"/>
-      <parent link="${prefix}base_link"/>
-      <child link="${prefix}top_right_camera"/>
+<!--    Add sensors-->
+<!-- top-right-camera -->
+    <xacro:pointgrey_flea3 name="top_right_camera" frame="top_right_camera"/>
+    <joint name="base_link_to_top_right_camera" type="fixed">
+      <origin xyz="${length_offset} -0.22 ${1.35+height_offset}" rpy="0 0.4 0"/>
+      <parent link="base_link"/>
+      <child link="top_right_camera"/>
     </joint>
     <!-- top-left-camera -->
-    <xacro:pointgrey_flea3 name="${prefix}top_left_camera" frame="${prefix}top_left_camera"/>
-    <joint name="${prefix}base_link_to_${prefix}top_left_camera" type="fixed">
-      <origin xyz="-1.55 0.22 1.35" rpy="0 0.4 0"/>
-      <parent link="${prefix}base_link"/>
-      <child link="${prefix}top_left_camera"/>
+    <xacro:pointgrey_flea3 name="top_left_camera" frame="top_left_camera"/>
+    <joint name="base_link_to_top_left_camera" type="fixed">
+      <origin xyz="${length_offset} 0.22 ${1.35+height_offset}" rpy="0 0.4 0"/>
+      <parent link="base_link"/>
+      <child link="top_left_camera"/>
     </joint>
-    <!-- laser sensor lms_ldmrs400001 -->
-    <xacro:sick_ldmrs name="${prefix}frontal_laser"/>
-    <joint name="${prefix}base_link_to_${prefix}frontal_laser_mount_link" type="fixed">
-      <origin xyz="0 0 0" rpy="0 0 0"/>
-      <parent link="${prefix}base_link"/>
-      <child link="${prefix}frontal_laser_mount_link"/>
-    </joint>
-    <!-- left lms151 laser -->
-    <xacro:sick_lms1xx frame="${prefix}right_laser"/>
-    <joint name="${prefix}base_link_to_${prefix}right_laser" type="fixed">
-      <origin xyz="-0.07 -0.76 0.27" rpy="0 0 ${-0.7854}"/>
-      <parent link="${prefix}base_link"/>
-      <child link="${prefix}right_laser"/>
-    </joint>
-    <!-- right lms151 laser -->
-    <xacro:sick_lms1xx frame="${prefix}left_laser"/>
-    <joint name="${prefix}base_link_to_${prefix}left_laser" type="fixed">
-      <origin xyz="-0.07 0.76  0.27" rpy="0 0 ${0.7854}"/>
-      <parent link="${prefix}base_link"/>
-      <child link="${prefix}left_laser"/>
-    </joint>
-    <!-- RGB-D camera -->
-    <xacro:asus_camera_model name="${prefix}top_center_rgbd_camera"/>
-    <joint name="${prefix}base_link_to_${prefix}top_center_rgbd_camera" type="fixed">
-      <!--            <origin xyz="-1.510 -0.010 1.397" rpy="-0.000 0.223 -0.000" />-->
-      <origin xyz="-1.510 -0.010 1.338" rpy="-0.000 0.207 -0.000"/>
-      <!--            <origin xyz="-1.51 -0.01 1.27" rpy="0 0.4 0" />-->
-      <parent link="${prefix}base_link"/>
-      <child link="${prefix}top_center_rgbd_camera_link"/>
-    </joint>
-  </xacro:macro>
-      <!-- Call the xacro macro-->
-    <xacro:atlascar2 prefix=""/>
+    <!-- top velodyne lidar -->
+    <xacro:VLP-16 name="VLP_lidar" parent="base_link" topic="/lidar_1/velodyne_points">
+      <origin xyz="0 0 ${1.35+height_offset}" rpy="0 0 0"/>
+    </xacro:VLP-16>
+    <!-- joints for ackermann_steering_controller -->
+    <xacro:front_steer name="front" parent="base" radius="${wheel_radius}" thickness="${thickness}"
+                       length="${length}" width="${width}" axel_offset="${axel_offset_x}" steer_height="${wheel_radius+steer_offset}">
+        <origin xyz="${length/2-axel_offset_x} 0 0" rpy="${-90 * deg_to_rad} 0 ${90 * deg_to_rad}"/>
+    </xacro:front_steer>
+    <xacro:rear_wheel name="rear" parent="base" radius="${wheel_radius}" thickness="${thickness}">
+        <origin xyz="${-length/2+axel_offset_x} 0 0" rpy="${-90 * deg_to_rad} 0 ${-90 * deg_to_rad}"/>
+    </xacro:rear_wheel>
+    <!-- Wheels -->
+    <xacro:front_wheel_lr name="front_right" parent="base" radius="${wheel_radius}" thickness="${thickness}"
+                          length="${length}" width="${width}" axel_offset="${axel_offset_x}" right_left="1" steer_height="${wheel_radius+steer_offset}">
+        <origin xyz="${length/2-axel_offset_x} ${width/2+axel_offset_y} 0" rpy="${-90 * deg_to_rad} 0 0"/>
+    </xacro:front_wheel_lr>
+    <xacro:front_wheel_lr name="front_left" parent="base" radius="${wheel_radius}" thickness="${thickness}"
+                          length="${length}" width="${width}" axel_offset="${axel_offset_x}" right_left="-1" steer_height="${wheel_radius+steer_offset}">
+        <origin xyz="${length/2-axel_offset_x} ${-width/2-axel_offset_y} 0" rpy="${-90 * deg_to_rad} 0 0"/>
+    </xacro:front_wheel_lr>
+    <xacro:rear_wheel_lr name="rear_right" parent="base" radius="${wheel_radius}" right_left="1" thickness="${thickness}">
+        <origin xyz="${-length/2+axel_offset_x - 0.05} ${width/2+axel_offset_y} 0" rpy="${-90 * deg_to_rad} 0 ${-90 * deg_to_rad}"/>
+    </xacro:rear_wheel_lr>
+    <xacro:rear_wheel_lr name="rear_left" parent="base" radius="${wheel_radius}" right_left="-1" thickness="${thickness}">
+        <origin xyz="${-length/2+axel_offset_x - 0.05} ${-width/2-axel_offset_y} 0" rpy="${-90 * deg_to_rad} 0 ${90 * deg_to_rad}"/>
+    </xacro:rear_wheel_lr>
+    <!-- Gazebo plugin for ROS Control -->
+    <gazebo>
+        <plugin name="gazebo_ros_control" filename="libgazebo_ros_control.so">
+            <robotSimType>steer_bot_hardware_gazebo/SteerBotHardwareGazebo</robotSimType>
+        </plugin>
+    </gazebo>
+    <!-- Colour -->
+    <gazebo reference="base_footprint">
+        <material>Gazebo/Purple</material>
+    </gazebo>
 </robot>

File: atlascar2_description/urdf/atlascar2_ackermann.urdf.xacro (robot description, xacro)
@@ -4,5 +4,5 @@
     Robot model taken from http://wiki.ros.org/pr2_mechanism/Tutorials/SImple%20URDF-Controller%20Example
     -->
-    <xacro:include filename="atlascar2_wheel.urdf.xacro"/>
+    <xacro:include filename="$(find atlascar2_description)/urdf/atlascar2_wheel.urdf.xacro"/>
     <xacro:include filename="$(find pointgrey_camera_description)/urdf/pointgrey_flea3.urdf.xacro"/>
     <xacro:include filename="$(find sick_ldmrs_description)/urdf/sick_ldmrs_macros.urdf.xacro"/>

File: atlascar2_description/urdf/atlascar2_ackermann_VLP.urdf.xacro (robot description, xacro)
@@ -4,5 +4,5 @@
     Robot model taken from http://wiki.ros.org/pr2_mechanism/Tutorials/SImple%20URDF-Controller%20Example
     -->
-    <xacro:include filename="atlascar2_wheel.urdf.xacro"/>
+    <xacro:include filename="$(find atlascar2_description)/urdf/atlascar2_wheel.urdf.xacro"/>
     <xacro:include filename="$(find pointgrey_camera_description)/urdf/pointgrey_flea3.urdf.xacro"/>
     <xacro:include filename="$(find velodyne_description)/urdf/VLP-16.urdf.xacro"/>

Commit message: #32 lardemua/atom#425 New try at configuration with a similar error

File: atlascar2_calibration/urdf/initial_estimate.urdf.xacro (robot description, xacro)
@@ -7,4 +7,7 @@
     <xacro:include filename="$(find pointgrey_camera_description)/urdf/pointgrey_flea3.urdf.xacro"/>
     <xacro:include filename="$(find velodyne_description)/urdf/VLP-16.urdf.xacro"/>
+    <xacro:include filename="$(find pointgrey_camera_description)/urdf/pointgrey_flea3.urdf.xacro"/>
+    <!-- <xacro:include filename="$(find sick_ldmrs_description)/urdf/sick_ldmrs_macros.urdf.xacro"/> -->
+    <xacro:include filename="$(find lms1xx)/urdf/sick_lms1xx.urdf.xacro"/>
     <xacro:property name="deg_to_rad" value="0.01745329251994329577"/>
     <!-- Constants for robot dimensions -->
@@ -20,4 +23,5 @@
     <xacro:property name="axel_offset_y" value="0" /> <!-- Space btw top of beam and the each joint -->
     <xacro:property name="steer_offset" value="0.02" /> <!-- Link 1 -->
+    <xacro:property name="vehicle_name" value="atlascar2"/> <!-- Name of vehicle-->
     <!-- Links: inertial,visual,collision -->
     <link name="base_link">
@@ -86,5 +90,5 @@
     </joint>
     <!-- top velodyne lidar -->
-    <xacro:VLP-16 name="VLP_lidar" parent="base_link" topic="/lidar_1/velodyne_points">
+    <xacro:VLP-16 name="top_laser" parent="base_link" topic="top_laser/cloud">
       <origin xyz="0 0 ${1.35+height_offset}" rpy="0 0 0"/>
     </xacro:VLP-16>
@@ -97,4 +101,25 @@
         <origin xyz="${-length/2+axel_offset_x} 0 0" rpy="${-90 * deg_to_rad} 0 ${-90 * deg_to_rad}"/>
     </xacro:rear_wheel>
+    <!-- laser sensor lms_ldmrs400001 -->
+    <!-- <xacro:sick_ldmrs name="frontal_laser"/> -->
+    <!-- <joint name="base_link_to_frontal_laser_mount_link" type="fixed"> -->
+      <!-- <origin xyz="${length/2 + length_offset} 0 ${height_offset}" rpy="0 0 0"/> -->
+      <!-- <parent link="base_link"/> -->
+      <!-- <child link="frontal_laser_mount_link"/> -->
+    <!-- </joint> -->
+    <!-- left lms151 laser -->
+    <xacro:sick_lms1xx frame="left_laser" topic="/atlascar2/left_laser/scan"/>
+    <joint name="base_link_to_left_laser" type="fixed">
+      <origin xyz="${length/2 + length_offset - 0.08} 0.76 ${height_offset+0.27}" rpy="0 0 ${0.7854}"/>
+      <parent link="base_link"/>
+      <child link="left_laser"/>
+    </joint>
+    <!-- right lms151 laser -->
+    <xacro:sick_lms1xx frame="right_laser" topic="/atlascar2/right_laser/scan"/>
+    <joint name="base_link_to_right_laser" type="fixed">
+      <origin xyz="${length/2 + length_offset - 0.08} -0.76 ${height_offset+0.27}" rpy="0 0 ${-0.7854}"/>
+      <parent link="base_link"/>
+      <child link="right_laser"/>
+    </joint>
     <!-- Wheels -->
     <xacro:front_wheel_lr name="front_right" parent="base" radius="${wheel_radius}" thickness="${thickness}"

File: atlascar2_description/urdf/atlascar2_ackermann_VLP.urdf.xacro (robot description, xacro)
@@ -8,5 +8,5 @@
     <xacro:include filename="$(find velodyne_description)/urdf/VLP-16.urdf.xacro"/>
     <xacro:include filename="$(find pointgrey_camera_description)/urdf/pointgrey_flea3.urdf.xacro"/>
-    <xacro:include filename="$(find sick_ldmrs_description)/urdf/sick_ldmrs_macros.urdf.xacro"/>
+    <!-- <xacro:include filename="$(find sick_ldmrs_description)/urdf/sick_ldmrs_macros.urdf.xacro"/> -->
     <xacro:include filename="$(find lms1xx)/urdf/sick_lms1xx.urdf.xacro"/>
     <xacro:property name="deg_to_rad" value="0.01745329251994329577"/>
@@ -23,4 +23,5 @@
     <xacro:property name="axel_offset_y" value="0" /> <!-- Space btw top of beam and the each joint -->
     <xacro:property name="steer_offset" value="0.02" /> <!-- Link 1 -->
+    <xacro:property name="vehicle_name" value="atlascar2"/> <!-- Name of vehicle-->
     <!-- Links: inertial,visual,collision -->
     <link name="base_link">
@@ -89,5 +90,5 @@
     </joint>
     <!-- top velodyne lidar -->
-    <xacro:VLP-16 name="top_lidar" parent="base_link" topic="/top_laser/cloud">
+    <xacro:VLP-16 name="top_laser" parent="base_link" topic="top_laser/cloud">
       <origin xyz="0 0 ${1.35+height_offset}" rpy="0 0 0"/>
     </xacro:VLP-16>
@@ -101,12 +102,12 @@
     </xacro:rear_wheel>
     <!-- laser sensor lms_ldmrs400001 -->
-    <xacro:sick_ldmrs name="frontal_laser"/>
-    <joint name="base_link_to_frontal_laser_mount_link" type="fixed">
-      <origin xyz="${length/2 + length_offset} 0 ${height_offset}" rpy="0 0 0"/>
-      <parent link="base_link"/>
-      <child link="frontal_laser_mount_link"/>
-    </joint>
+    <!-- <xacro:sick_ldmrs name="frontal_laser"/> -->
+    <!-- <joint name="base_link_to_frontal_laser_mount_link" type="fixed"> -->
+      <!-- <origin xyz="${length/2 + length_offset} 0 ${height_offset}" rpy="0 0 0"/> -->
+      <!-- <parent link="base_link"/> -->
+      <!-- <child link="frontal_laser_mount_link"/> -->
+    <!-- </joint> -->
     <!-- left lms151 laser -->
-    <xacro:sick_lms1xx frame="left_laser" topic="/left_laser/scan"/>
+    <xacro:sick_lms1xx frame="left_laser" topic="/atlascar2/left_laser/scan"/>
     <joint name="base_link_to_left_laser" type="fixed">
       <origin xyz="${length/2 + length_offset - 0.08} 0.76 ${height_offset+0.27}" rpy="0 0 ${0.7854}"/>
@@ -115,5 +116,5 @@
     </joint>
     <!-- right lms151 laser -->
-    <xacro:sick_lms1xx frame="right_laser" topic="/right_laser/scan"/>
+    <xacro:sick_lms1xx frame="right_laser" topic="/atlascar2/right_laser/scan"/>
     <joint name="base_link_to_right_laser" type="fixed">
       <origin xyz="${length/2 + length_offset - 0.08} -0.76 ${height_offset+0.27}" rpy="0 0 ${-0.7854}"/>

Commit message: #32 lardemua/atom#425 Problem solved, data collection carries on as it should be

File: atlascar2_calibration/urdf/initial_estimate.urdf.xacro (robot description, xacro)
@@ -5,9 +5,7 @@
     -->
     <xacro:include filename="$(find atlascar2_description)/urdf/atlascar2_wheel.urdf.xacro"/>
-    <xacro:include filename="$(find pointgrey_camera_description)/urdf/pointgrey_flea3.urdf.xacro"/>
+    <xacro:include filename="$(find atlascar2_description)/urdf/atlascar2_ackermann.macro.urdf.xacro"/>
     <xacro:include filename="$(find velodyne_description)/urdf/VLP-16.urdf.xacro"/>
-    <xacro:include filename="$(find pointgrey_camera_description)/urdf/pointgrey_flea3.urdf.xacro"/>
     <!-- <xacro:include filename="$(find sick_ldmrs_description)/urdf/sick_ldmrs_macros.urdf.xacro"/> -->
-    <xacro:include filename="$(find lms1xx)/urdf/sick_lms1xx.urdf.xacro"/>
     <xacro:property name="deg_to_rad" value="0.01745329251994329577"/>
     <!-- Constants for robot dimensions -->
@@ -24,69 +22,15 @@
     <xacro:property name="steer_offset" value="0.02" /> <!-- Link 1 -->
     <xacro:property name="vehicle_name" value="atlascar2"/> <!-- Name of vehicle-->
-    <!-- Links: inertial,visual,collision -->
-    <link name="base_link">
-        <inertial>
-            <!-- origin is relative -->
-            <origin xyz="0 0 0" rpy="0 0 0"/>
-            <mass value="2"/>
-            <inertia ixx="1" ixy="0" ixz="0"
-                     iyy="1" iyz="0"
-                     izz="1"/>
-        </inertial>
-        <visual>
-            <origin xyz=" ${length/2} ${-width/2 - 0.15} ${-wheel_radius + 0.05}" rpy="0 0 ${90*deg_to_rad}"/>
-            <geometry>
-                <mesh filename="file:///$(find atlascar2_description)/meshes/atlascar2_nowheels.dae"/>
-            </geometry>
-        </visual>
-        <collision>
-            <!-- origin is relative -->
-            <origin xyz=" 0 0 ${-wheel_radius + height/2}"/>
-            <geometry>
-                <box size="${length - 0.1} ${width} ${height/2}"/>
-            </geometry>
-        </collision>
-    </link>
-    <link name="top_collision">
-        <collision>
-            <origin xyz="${-length/7} 0 0"/>
-            <geometry>
-                <box size="${length/2} ${width} ${height/2}"/>
-            </geometry>
-        </collision>
-    </link>
-    <joint name="base_link_to_top_collision" type="fixed">
-        <origin xyz="0 0 ${height/2}" rpy="0 0 0"/>
-        <parent link="base_link"/>
-        <child link="top_collision"/>
-    </joint>
-    <link name="base_footprint">
-        <collision>
-            <origin xyz="0 0 0"/>
-            <geometry>
-                <sphere radius="0.00000001"/>
-            </geometry>
-        </collision>
-    </link>
-    <joint name="base_footprint_joint" type="fixed">
-        <origin xyz="0 0 ${wheel_radius}" rpy="0 0 0"/>
-        <child link="base_link"/>
-        <parent link="base_footprint"/>
-    </joint>
-<!--    Add sensors-->
-<!-- top-right-camera -->
-    <xacro:pointgrey_flea3 name="top_right_camera" frame="top_right_camera"/>
-    <joint name="base_link_to_top_right_camera" type="fixed">
-      <origin xyz="${length_offset} -0.22 ${1.35+height_offset}" rpy="0 0.4 0"/>
-      <parent link="base_link"/>
-      <child link="top_right_camera"/>
-    </joint>
+    <!-- Add car macro -->
+    <xacro:atlascar2 length="${length}" width="${width}" height="${height}" wheel_radius="${wheel_radius}"/>
+    <!--    Add sensors-->
+    <!-- top-right-camera -->
+    <xacro:pointgrey_flea3_joints name="top_right_camera" frame="top_right_camera" parent="base_link"
+                                  x="${length_offset}" y="-0.22" z="${1.35+height_offset}"
+                                  rol="0" pit="0.4" yaw="0"/>
     <!-- top-left-camera -->
-    <xacro:pointgrey_flea3 name="top_left_camera" frame="top_left_camera"/>
-    <joint name="base_link_to_top_left_camera" type="fixed">
-      <origin xyz="${length_offset} 0.22 ${1.35+height_offset}" rpy="0 0.4 0"/>
-      <parent link="base_link"/>
-      <child link="top_left_camera"/>
-    </joint>
+    <xacro:pointgrey_flea3_joints name="top_left_camera" frame="top_left_camera" parent="base_link"
+                                  x="${length_offset}" y="0.22" z="${1.35+height_offset}"
+                                  rol="0" pit="0.4" yaw="0"/>
     <!-- top velodyne lidar -->
     <xacro:VLP-16 name="top_laser" parent="base_link" topic="top_laser/cloud">
@@ -109,17 +53,11 @@
     <!-- </joint> -->
     <!-- left lms151 laser -->
-    <xacro:sick_lms1xx frame="left_laser" topic="/atlascar2/left_laser/scan"/>
-    <joint name="base_link_to_left_laser" type="fixed">
-      <origin xyz="${length/2 + length_offset - 0.08} 0.76 ${height_offset+0.27}" rpy="0 0 ${0.7854}"/>
-      <parent link="base_link"/>
-      <child link="left_laser"/>
-    </joint>
+    <xacro:sick_lms1xx_joints frame="left_laser" topic="/left_laser/scan" parent="base_link"
+                                  x="${length/2 + length_offset - 0.08}" y="0.76" z="${0.27+height_offset}"
+                                  rol="0" pit="0" yaw="0.7854"/>
     <!-- right lms151 laser -->
-    <xacro:sick_lms1xx frame="right_laser" topic="/atlascar2/right_laser/scan"/>
-    <joint name="base_link_to_right_laser" type="fixed">
-      <origin xyz="${length/2 + length_offset - 0.08} -0.76 ${height_offset+0.27}" rpy="0 0 ${-0.7854}"/>
-      <parent link="base_link"/>
-      <child link="right_laser"/>
-    </joint>
+    <xacro:sick_lms1xx_joints frame="right_laser" topic="/right_laser/scan" parent="base_link"
+                                  x="${length/2 + length_offset - 0.08}" y="-0.76" z="${0.27+height_offset}"
+                                  rol="0" pit="0" yaw="-0.7854"/>
     <!-- Wheels -->
     <xacro:front_wheel_lr name="front_right" parent="base" radius="${wheel_radius}" thickness="${thickness}"
