Commit message: #41 Bugfixing in visual odometry

File: atlascar2_calibration/urdf/optimized.urdf.xacro (robot description, xacro)
@@ -14,5 +14,5 @@
     </visual>
     <collision>
-      <origin xyz="0.0 0.0 0.52" rpy="0 0 0"/>
+      <origin xyz="0.0 0.0 0.52" rpy="0.0 0.0 0.0"/>
       <geometry>
         <box size="3.375 1.475 0.805"/>
@@ -22,5 +22,5 @@
   <link name="top_collision">
     <collision>
-      <origin xyz="-0.49642857142857144 0.0 0.0" rpy="0 0 0"/>
+      <origin xyz="-0.49642857142857144 0.0 0.0" rpy="0.0 0.0 0.0"/>
       <geometry>
         <box size="1.7375 1.475 0.805"/>
@@ -35,5 +35,5 @@
   <link name="base_footprint">
     <collision>
-      <origin xyz="0.0 0.0 0.0" rpy="0 0 0"/>
+      <origin xyz="0.0 0.0 0.0" rpy="0.0 0.0 0.0"/>
       <geometry>
         <sphere radius="1e-08"/>
@@ -110,5 +110,5 @@
   </gazebo>
   <joint name="{parent}_to_top_right_camera" type="fixed">
-    <origin xyz="0.2001221309726634 -0.21610799787967408 1.3694008135553515" rpy="-0.00033517103954637626 0.4008436654743302 -0.00044685990488837183"/>
+    <origin xyz="-0.021897489171257133 -0.43407180592799444 1.4630116543485698" rpy="-0.009651423175084316 0.23983548468788154 -0.07894715051412995"/>
     <parent link="base_link"/>
     <child link="top_right_camera"/>
@@ -178,10 +178,10 @@
   </gazebo>
   <joint name="{parent}_to_top_left_camera" type="fixed">
-    <origin xyz="0.20154699446691582 0.22553233689317445 1.368941444270171" rpy="-0.00033785773814485546 0.400753678202867 -0.0010168019601629586"/>
+    <origin xyz="0.26141185208258183 0.19623646085522287 1.4972876969069215" rpy="-0.015755168155665775 0.2870706091612352 -0.13638404608332255"/>
     <parent link="base_link"/>
     <child link="top_left_camera"/>
   </joint>
   <joint name="top_laser_base_mount_joint" type="fixed">
-    <origin xyz="0.0018114097858342693 0.006131485845022701 1.3555173396460185" rpy="0.0010523513027342205 -0.004039523504586624 -0.0014120572320113396"/>
+    <origin xyz="-0.04657862396873688 -0.004175433925296066 1.613198836396312" rpy="0.0029580079086952743 0.29858170602628203 -0.009716093302018955"/>
     <parent link="base_link"/>
     <child link="top_laser_base_link"/>
@@ -189,5 +189,5 @@
   <link name="top_laser_base_link">
     <inertial>
-      <origin xyz="0.0 0.0 0.03585" rpy="0 0 0"/>
+      <origin xyz="0.0 0.0 0.03585" rpy="0.0 0.0 0.0"/>
       <mass value="0.83"/>
       <inertia ixx="0.000908059425" ixy="0.0" ixz="0.0" iyy="0.000908059425" iyz="0.0" izz="0.0011049624"/>
@@ -217,10 +217,10 @@
   <link name="top_laser">
     <inertial>
-      <origin xyz="0.0 0.0 0.0" rpy="0 0 0"/>
+      <origin xyz="0.0 0.0 0.0" rpy="0.0 0.0 0.0"/>
       <mass value="0.01"/>
       <inertia ixx="1e-07" ixy="0.0" ixz="0.0" iyy="1e-07" iyz="0.0" izz="1e-07"/>
     </inertial>
     <visual>
-      <origin xyz="0.0 0.0 -0.0377" rpy="0 0 0"/>
+      <origin xyz="0.0 0.0 -0.0377" rpy="0.0 0.0 0.0"/>
       <geometry>
         <mesh filename="package://velodyne_description/meshes/VLP16_scan.dae"/>
@@ -272,6 +272,6 @@
     <inertial>
       <origin xyz="0.0 0.0 0.0" rpy="0.0 0.0 0.0"/>
-      <mass value="0.3"/>
-      <inertia ixx="0.02" ixy="0.0" ixz="0.0" iyy="0.002" iyz="0.0" izz="0.02"/>
+      <mass value="11.16"/>
+      <inertia ixx="0.246171" ixy="0.0" ixz="0.0" iyy="0.246171" iyz="0.0" izz="0.4532354999999999"/>
     </inertial>
     <collision>
@@ -303,6 +303,6 @@
     <inertial>
       <origin xyz="0.0 0.0 0.0" rpy="0.0 0.0 0.0"/>
-      <mass value="0.3"/>
-      <inertia ixx="0.02" ixy="0.0" ixz="0.0" iyy="0.002" iyz="0.0" izz="0.02"/>
+      <mass value="11.16"/>
+      <inertia ixx="0.246171" ixy="0.0" ixz="0.0" iyy="0.246171" iyz="0.0" izz="0.4532354999999999"/>
     </inertial>
     <collision>
@@ -329,5 +329,5 @@
   <link name="left_laser">
     <inertial>
-      <origin xyz="0.0 0.0 0.0" rpy="0 0 0"/>
+      <origin xyz="0.0 0.0 0.0" rpy="0.0 0.0 0.0"/>
       <mass value="1.1"/>
       <inertia ixx="0.00307156543804" ixy="0.0" ixz="0.0" iyy="0.0031284904152700005" iyz="0.0" izz="0.00196432421427"/>
@@ -386,5 +386,5 @@
   <link name="right_laser">
     <inertial>
-      <origin xyz="0.0 0.0 0.0" rpy="0 0 0"/>
+      <origin xyz="0.0 0.0 0.0" rpy="0.0 0.0 0.0"/>
       <mass value="1.1"/>
       <inertia ixx="0.00307156543804" ixy="0.0" ixz="0.0" iyy="0.0031284904152700005" iyz="0.0" izz="0.00196432421427"/>
@@ -444,6 +444,6 @@
     <inertial>
       <origin xyz="0.0 0.0 0.0" rpy="0.0 0.0 0.0"/>
-      <mass value="0.3"/>
-      <inertia ixx="0.02" ixy="0.0" ixz="0.0" iyy="0.002" iyz="0.0" izz="0.02"/>
+      <mass value="11.16"/>
+      <inertia ixx="0.246171" ixy="0.0" ixz="0.0" iyy="0.246171" iyz="0.0" izz="0.4532354999999999"/>
     </inertial>
     <collision>
@@ -465,6 +465,6 @@
     <inertial>
       <origin xyz="0.0 0.0 0.0" rpy="0.0 0.0 0.0"/>
-      <mass value="0.3"/>
-      <inertia ixx="0.02" ixy="0.0" ixz="0.0" iyy="0.002" iyz="0.0" izz="0.02"/>
+      <mass value="11.16"/>
+      <inertia ixx="0.246171" ixy="0.0" ixz="0.0" iyy="0.246171" iyz="0.0" izz="0.4532354999999999"/>
     </inertial>
     <visual>
@@ -505,6 +505,6 @@
     <inertial>
       <origin xyz="0.0 0.0 0.0" rpy="0.0 0.0 0.0"/>
-      <mass value="0.3"/>
-      <inertia ixx="0.02" ixy="0.0" ixz="0.0" iyy="0.002" iyz="0.0" izz="0.02"/>
+      <mass value="11.16"/>
+      <inertia ixx="0.246171" ixy="0.0" ixz="0.0" iyy="0.246171" iyz="0.0" izz="0.4532354999999999"/>
     </inertial>
     <collision>
@@ -526,6 +526,6 @@
     <inertial>
       <origin xyz="0.0 0.0 0.0" rpy="0.0 0.0 0.0"/>
-      <mass value="0.3"/>
-      <inertia ixx="0.02" ixy="0.0" ixz="0.0" iyy="0.002" iyz="0.0" izz="0.02"/>
+      <mass value="11.16"/>
+      <inertia ixx="0.246171" ixy="0.0" ixz="0.0" iyy="0.246171" iyz="0.0" izz="0.4532354999999999"/>
     </inertial>
     <visual>
@@ -566,6 +566,6 @@
     <inertial>
       <origin xyz="0.0 0.0 0.0" rpy="0.0 0.0 0.0"/>
-      <mass value="0.3"/>
-      <inertia ixx="0.02" ixy="0.0" ixz="0.0" iyy="0.002" iyz="0.0" izz="0.02"/>
+      <mass value="11.16"/>
+      <inertia ixx="0.246171" ixy="0.0" ixz="0.0" iyy="0.246171" iyz="0.0" izz="0.4532354999999999"/>
     </inertial>
     <visual>
@@ -599,6 +599,6 @@
     <inertial>
       <origin xyz="0.0 0.0 0.0" rpy="0.0 0.0 0.0"/>
-      <mass value="0.3"/>
-      <inertia ixx="0.02" ixy="0.0" ixz="0.0" iyy="0.002" iyz="0.0" izz="0.02"/>
+      <mass value="11.16"/>
+      <inertia ixx="0.246171" ixy="0.0" ixz="0.0" iyy="0.246171" iyz="0.0" izz="0.4532354999999999"/>
     </inertial>
     <visual>
