Commit message: .

File: atlascar2_calibration/urdf/initial_estimate.urdf.xacro (robot description, xacro)
@@ -1,639 +1,92 @@
-<?xml version="1.0" ?>
-<robot name="atlascar2" version="1.0">
-  <link name="base_link">
-    <inertial>
-      <origin xyz="0.0 0.0 0.0" rpy="0.0 0.0 0.0"/>
-      <mass value="2.0"/>
-      <inertia ixx="1.0" ixy="0.0" ixz="0.0" iyy="1.0" iyz="0.0" izz="1.0"/>
-    </inertial>
-    <visual>
-      <origin xyz="1.7375 -0.8875000000000001 -0.235" rpy="0.0 0.0 1.5707963267948966"/>
-      <geometry>
-        <mesh filename="file:////home/nel/catkin_ws/src/calibration/robots/atlascar2/atlascar2_description/meshes/atlascar2_nowheels.dae"/>
-      </geometry>
-    </visual>
-    <collision>
-      <origin xyz="0.0 0.0 0.52" rpy="0.0 0.0 0.0"/>
-      <geometry>
-        <box size="3.375 1.475 0.805"/>
-      </geometry>
-    </collision>
-  </link>
-  <link name="top_collision">
-    <collision>
-      <origin xyz="-0.49642857142857144 0.0 0.0" rpy="0.0 0.0 0.0"/>
-      <geometry>
-        <box size="1.7375 1.475 0.805"/>
-      </geometry>
-    </collision>
-  </link>
-  <joint name="base_link_to_top_collision" type="fixed">
-    <origin xyz="0.0 0.0 0.805" rpy="0.0 0.0 0.0"/>
-    <parent link="base_link"/>
-    <child link="top_collision"/>
-  </joint>
-  <link name="base_footprint">
-    <collision>
-      <origin xyz="0.0 0.0 0.0" rpy="0.0 0.0 0.0"/>
-      <geometry>
-        <sphere radius="1e-08"/>
-      </geometry>
-    </collision>
-  </link>
-  <joint name="base_footprint_joint" type="fixed">
-    <origin xyz="0.0 0.0 0.285" rpy="0.0 0.0 0.0"/>
-    <parent link="base_footprint"/>
-    <child link="base_link"/>
-  </joint>
-  <link name="top_right_camera">
-    <inertial>
-      <mass value="0.085"/>
-      <inertia ixx="1e-06" ixy="0.0" ixz="0.0" iyy="1e-06" iyz="0.0" izz="1e-06"/>
-    </inertial>
-    <visual>
-      <origin xyz="0.0 0.0 0.0" rpy="0.0 0.0 0.0"/>
-      <geometry>
-        <box size="0.0754 0.029 0.035"/>
-      </geometry>
-      <material name="dark_grey"/>
-    </visual>
-    <collision>
-      <origin xyz="0.0 0.0 0.0" rpy="0.0 0.0 0.0"/>
-      <geometry>
-        <box size="0.0754 0.029 0.035"/>
-      </geometry>
-    </collision>
-  </link>
-  <link name="top_right_camera_optical"/>
-  <joint name="top_right_camera_optical_joint" type="fixed">
-    <origin xyz="0.0 0.0 0.0" rpy="-1.570796 0.0 -1.570796"/>
-    <parent link="top_right_camera"/>
-    <child link="top_right_camera_optical"/>
-  </joint>
-  <gazebo reference="top_right_camera_optical">
-    <material>Gazebo/Grey</material>
-    <sensor name="top_right_camera" type="camera">
-      <update_rate>120</update_rate>
-      <camera name="top_right_camera">
-        <pose>0 0 0 0 -1.5707 1.5707</pose>
-        <horizontal_fov>1.0471975512</horizontal_fov>
-        <image>
-          <width>1272</width>
-          <height>1016</height>
-          <format>R8G8B8</format>
-        </image>
-        <clip>
-          <near>0.5</near>
-          <far>300</far>
-        </clip>
-        <noise>
-          <type>gaussian</type>
-          <mean>0.0</mean>
-          <stddev>0.007</stddev>
-        </noise>
-      </camera>
-      <plugin filename="libgazebo_ros_camera.so" name="camera_controller">
-        <alwaysOn>true</alwaysOn>
-        <updateRate>120</updateRate>
-        <cameraName>top_right_camera</cameraName>
-        <imageTopicName>image_raw</imageTopicName>
-        <cameraInfoTopicName>camera_info</cameraInfoTopicName>
-        <frameName>top_right_camera_optical</frameName>
-        <hackBaseline>0.07</hackBaseline>
-        <distortionK1>0.0</distortionK1>
-        <distortionK2>0.0</distortionK2>
-        <distortionK3>0.0</distortionK3>
-        <distortionT1>0.0</distortionT1>
-        <distortionT2>0.0</distortionT2>
-      </plugin>
-    </sensor>
-  </gazebo>
-  <joint name="{parent}_to_top_right_camera" type="fixed">
-    <origin xyz="0.20000000298023224 -0.31146225333213806 1.4500000476837158" rpy="0.0018889869443012857 0.21043392484409348 -0.08979193626631238"/>
-    <parent link="base_link"/>
-    <child link="top_right_camera"/>
-  </joint>
-  <link name="top_left_camera">
-    <inertial>
-      <mass value="0.085"/>
-      <inertia ixx="1e-06" ixy="0.0" ixz="0.0" iyy="1e-06" iyz="0.0" izz="1e-06"/>
-    </inertial>
-    <visual>
-      <origin xyz="0.0 0.0 0.0" rpy="0.0 0.0 0.0"/>
-      <geometry>
-        <box size="0.0754 0.029 0.035"/>
-      </geometry>
-      <material name="dark_grey"/>
-    </visual>
-    <collision>
-      <origin xyz="0.0 0.0 0.0" rpy="0.0 0.0 0.0"/>
-      <geometry>
-        <box size="0.0754 0.029 0.035"/>
-      </geometry>
-    </collision>
-  </link>
-  <link name="top_left_camera_optical"/>
-  <joint name="top_left_camera_optical_joint" type="fixed">
-    <origin xyz="0.0 0.0 0.0" rpy="-1.570796 0.0 -1.570796"/>
-    <parent link="top_left_camera"/>
-    <child link="top_left_camera_optical"/>
-  </joint>
-  <gazebo reference="top_left_camera_optical">
-    <material>Gazebo/Grey</material>
-    <sensor name="top_left_camera" type="camera">
-      <update_rate>120</update_rate>
-      <camera name="top_left_camera">
-        <pose>0 0 0 0 -1.5707 1.5707</pose>
-        <horizontal_fov>1.0471975512</horizontal_fov>
-        <image>
-          <width>1272</width>
-          <height>1016</height>
-          <format>R8G8B8</format>
-        </image>
-        <clip>
-          <near>0.5</near>
-          <far>300</far>
-        </clip>
-        <noise>
-          <type>gaussian</type>
-          <mean>0.0</mean>
-          <stddev>0.007</stddev>
-        </noise>
-      </camera>
-      <plugin filename="libgazebo_ros_camera.so" name="camera_controller">
-        <alwaysOn>true</alwaysOn>
-        <updateRate>120</updateRate>
-        <cameraName>top_left_camera</cameraName>
-        <imageTopicName>image_raw</imageTopicName>
-        <cameraInfoTopicName>camera_info</cameraInfoTopicName>
-        <frameName>top_left_camera_optical</frameName>
-        <hackBaseline>0.07</hackBaseline>
-        <distortionK1>0.0</distortionK1>
-        <distortionK2>0.0</distortionK2>
-        <distortionK3>0.0</distortionK3>
-        <distortionT1>0.0</distortionT1>
-        <distortionT2>0.0</distortionT2>
-      </plugin>
-    </sensor>
-  </gazebo>
-  <joint name="{parent}_to_top_left_camera" type="fixed">
-    <origin xyz="0.20000000298023224 0.2464757263660431 1.4500000476837158" rpy="0.013418349553578884 0.28826911184579374 -0.15358350614019278"/>
-    <parent link="base_link"/>
-    <child link="top_left_camera"/>
-  </joint>
-  <joint name="top_laser_base_mount_joint" type="fixed">
-    <origin xyz="0.2420397400856018 0.0 1.4409246444702148" rpy="1.4630187760947651e-08 0.20393157921432659 2.0505546692252536e-09"/>
-    <parent link="base_link"/>
-    <child link="top_laser_base_link"/>
-  </joint>
-  <link name="top_laser_base_link">
-    <inertial>
-      <origin xyz="0.0 0.0 0.03585" rpy="0.0 0.0 0.0"/>
-      <mass value="0.83"/>
-      <inertia ixx="0.000908059425" ixy="0.0" ixz="0.0" iyy="0.000908059425" iyz="0.0" izz="0.0011049624"/>
-    </inertial>
-    <visual>
-      <geometry>
-        <mesh filename="package://velodyne_description/meshes/VLP16_base_1.dae"/>
-      </geometry>
-    </visual>
-    <visual>
-      <geometry>
-        <mesh filename="package://velodyne_description/meshes/VLP16_base_2.dae"/>
-      </geometry>
-    </visual>
-    <collision>
-      <origin xyz="0.0 0.0 0.03585" rpy="0.0 0.0 0.0"/>
-      <geometry>
-        <cylinder radius="0.0516" length="0.0717"/>
-      </geometry>
-    </collision>
-  </link>
-  <joint name="top_laser_base_scan_joint" type="fixed">
-    <origin xyz="0.0 0.0 0.0377" rpy="0.0 0.0 0.0"/>
-    <parent link="top_laser_base_link"/>
-    <child link="top_laser"/>
-  </joint>
-  <link name="top_laser">
-    <inertial>
-      <origin xyz="0.0 0.0 0.0" rpy="0.0 0.0 0.0"/>
-      <mass value="0.01"/>
-      <inertia ixx="1e-07" ixy="0.0" ixz="0.0" iyy="1e-07" iyz="0.0" izz="1e-07"/>
-    </inertial>
-    <visual>
-      <origin xyz="0.0 0.0 -0.0377" rpy="0.0 0.0 0.0"/>
-      <geometry>
-        <mesh filename="package://velodyne_description/meshes/VLP16_scan.dae"/>
-      </geometry>
-    </visual>
-  </link>
-  <gazebo reference="top_laser">
-    <sensor name="top_laser-VLP16" type="ray">
-      <pose>0 0 0 0 0 0</pose>
-      <visualize>false</visualize>
-      <update_rate>10</update_rate>
-      <ray>
-        <scan>
-          <horizontal>
-            <samples>1875</samples>
-            <resolution>1</resolution>
-            <min_angle>-3.141592653589793</min_angle>
-            <max_angle>3.141592653589793</max_angle>
-          </horizontal>
-          <vertical>
-            <samples>16</samples>
-            <resolution>1</resolution>
-            <min_angle>-0.2617993877991494</min_angle>
-            <max_angle> 0.2617993877991494</max_angle>
-          </vertical>
-        </scan>
-        <range>
-          <min>0.3</min>
-          <max>131.0</max>
-          <resolution>0.001</resolution>
-        </range>
-        <noise>
-          <type>gaussian</type>
-          <mean>0.0</mean>
-          <stddev>0.0</stddev>
-        </noise>
-      </ray>
-      <plugin filename="libgazebo_ros_velodyne_laser.so" name="gazebo_ros_laser_controller">
-        <topicName>top_laser/cloud</topicName>
-        <frameName>top_laser</frameName>
-        <organize_cloud>False</organize_cloud>
-        <min_range>0.9</min_range>
-        <max_range>130.0</max_range>
-        <gaussianNoise>0.008</gaussianNoise>
-      </plugin>
-    </sensor>
-  </gazebo>
-  <link name="front_steer_link">
-    <inertial>
-      <origin xyz="0.0 0.0 0.0" rpy="0.0 0.0 0.0"/>
-      <mass value="11.16"/>
-      <inertia ixx="0.246171" ixy="0.0" ixz="0.0" iyy="0.246171" iyz="0.0" izz="0.4532354999999999"/>
-    </inertial>
-    <collision>
-      <origin xyz="0.0 0.0 0.0" rpy="0.0 0.0 0.0"/>
-      <geometry>
-        <cylinder radius="0.05" length="0.02"/>
-      </geometry>
-    </collision>
-  </link>
-  <joint name="front_steer_joint" type="revolute">
-    <origin xyz="1.2375 0.0 0.305" rpy="0.0 0.0 0.0"/>
-    <axis xyz="0.0 0.0 1.0"/>
-    <parent link="base_link"/>
-    <child link="front_steer_link"/>
-    <limit effort="15.0" lower="-3.141592653589793" upper="3.141592653589793" velocity="5.0"/>
-    <dynamics damping="0.0" friction="0.0"/>
-  </joint>
-  <transmission name="front_steer_joint_trans">
-    <type>transmission_interface/SimpleTransmission</type>
-    <actuator name="front_steer_joint_motor"/>
-    <joint name="front_steer_joint">
-      <hardwareInterface>hardware_interface/PositionJointInterface</hardwareInterface>
-    </joint>
-  </transmission>
-  <gazebo reference="front_steer_link">
-    <material>Gazebo/Yellow</material>
-  </gazebo>
-  <link name="rear_wheel_link">
-    <inertial>
-      <origin xyz="0.0 0.0 0.0" rpy="0.0 0.0 0.0"/>
-      <mass value="11.16"/>
-      <inertia ixx="0.246171" ixy="0.0" ixz="0.0" iyy="0.246171" iyz="0.0" izz="0.4532354999999999"/>
-    </inertial>
-    <collision>
-      <origin xyz="0.0 0.0 0.0" rpy="0.0 0.0 0.0"/>
-      <geometry>
-        <cylinder radius="0.0028499999999999997" length="0.00145"/>
-      </geometry>
-    </collision>
-  </link>
-  <joint name="rear_wheel_joint" type="continuous">
-    <origin xyz="-1.2375 0.0 0.0" rpy="-1.5707963267948966 0.0 -1.5707963267948966"/>
-    <axis xyz="1.0 0.0 0.0"/>
-    <parent link="base_link"/>
-    <child link="rear_wheel_link"/>
-    <dynamics damping="0.0" friction="0.0"/>
-  </joint>
-  <transmission name="rear_wheel_joint_trans">
-    <type>transmission_interface/SimpleTransmission</type>
-    <actuator name="rear_wheel_joint_motor"/>
-    <joint name="rear_wheel_joint">
-      <hardwareInterface>hardware_interface/VelocityJointInterface</hardwareInterface>
-    </joint>
-  </transmission>
-  <link name="left_laser">
-    <inertial>
-      <origin xyz="0.0 0.0 0.0" rpy="0.0 0.0 0.0"/>
-      <mass value="1.1"/>
-      <inertia ixx="0.00307156543804" ixy="0.0" ixz="0.0" iyy="0.0031284904152700005" iyz="0.0" izz="0.00196432421427"/>
-    </inertial>
-    <visual>
-      <origin xyz="0.0 0.0 0.0" rpy="0.0 0.0 0.0"/>
-      <geometry>
-        <mesh filename="package://lms1xx/meshes/sick-lms1xx.dae"/>
-      </geometry>
-    </visual>
-    <collision>
-      <origin xyz="0.0 0.0 -0.05" rpy="0.0 0.0 0.0"/>
-      <geometry>
-        <box size="0.105 0.1 0.1"/>
-      </geometry>
-    </collision>
-  </link>
-  <gazebo reference="left_laser">
-    <turnGravityOff>true</turnGravityOff>
-    <sensor name="left_laser" type="ray">
-      <pose>0 0 0 0 0 0</pose>
-      <visualize>false</visualize>
-      <update_rate>50</update_rate>
-      <ray>
-        <scan>
-          <horizontal>
-            <samples>720</samples>
-            <resolution>1</resolution>
-            <min_angle>-2.35619</min_angle>
-            <max_angle>2.35619</max_angle>
-          </horizontal>
-        </scan>
-        <range>
-          <min>0.1</min>
-          <max>30.0</max>
-          <resolution>0.01</resolution>
-        </range>
-        <noise>
-          <type>gaussian</type>
-          <mean>0.0</mean>
-          <stddev>0.001</stddev>
-        </noise>
-      </ray>
-      <plugin filename="libgazebo_ros_laser.so" name="gazebo_ros_laser">
-        <topicName>/left_laser/scan</topicName>
-        <frameName>left_laser</frameName>
-        <robotNamespace>/</robotNamespace>
-      </plugin>
-    </sensor>
-  </gazebo>
-  <joint name="{parent}_to_left_laser" type="fixed">
-    <origin xyz="1.8575 0.76 0.37" rpy="0.0 0.0 0.7854"/>
-    <parent link="base_link"/>
-    <child link="left_laser"/>
-  </joint>
-  <link name="right_laser">
-    <inertial>
-      <origin xyz="0.0 0.0 0.0" rpy="0.0 0.0 0.0"/>
-      <mass value="1.1"/>
-      <inertia ixx="0.00307156543804" ixy="0.0" ixz="0.0" iyy="0.0031284904152700005" iyz="0.0" izz="0.00196432421427"/>
-    </inertial>
-    <visual>
-      <origin xyz="0.0 0.0 0.0" rpy="0.0 0.0 0.0"/>
-      <geometry>
-        <mesh filename="package://lms1xx/meshes/sick-lms1xx.dae"/>
-      </geometry>
-    </visual>
-    <collision>
-      <origin xyz="0.0 0.0 -0.05" rpy="0.0 0.0 0.0"/>
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
File: atlascar2_calibration/urdf/optimized_w_pattern.urdf.xacro (robot description, xacro)
@@ -45,4 +45,10 @@
     <parent link="base_footprint"/>
     <child link="base_link"/>
+  </joint>
+  <link name="world"/>
+  <joint name="world_to_base_footprint" type="fixed">
+    <origin xyz="0.0 0.0 0.0" rpy="0.0 0.0 0.0"/>
+    <parent link="world"/>
+    <child link="base_footprint"/>
   </joint>
   <link name="top_right_camera">
@@ -110,5 +116,5 @@
   </gazebo>
   <joint name="{parent}_to_top_right_camera" type="fixed">
-    <origin xyz="0.20428410540814848 -0.22388230247232627 1.447061150205553" rpy="-0.00042622049778580357 0.3988143668006885 -0.3"/>
+    <origin xyz="-2.506966815113514 -0.3112282304999219 1.6544852784893538" rpy="0.7446243395800726 0.390989048771717 0.12294531445427181"/>
     <parent link="base_link"/>
     <child link="top_right_camera"/>
@@ -178,10 +184,10 @@
   </gazebo>
   <joint name="{parent}_to_top_left_camera" type="fixed">
-    <origin xyz="0.20000000000000043 0.22000000000000017 1.4500000000000002" rpy="-1.5554606490236454e-16 0.4 0.3"/>
+    <origin xyz="-2.609787616289452 0.2802627642559952 1.8279500114804843" rpy="0.69396180745709 0.3040098754709762 0.1324511238181686"/>
     <parent link="base_link"/>
     <child link="top_left_camera"/>
   </joint>
   <joint name="top_laser_base_mount_joint" type="fixed">
-    <origin xyz="0.016363087328487538 0.01008967362563249 1.4746227815305066" rpy="-0.0022630437000740813 0.010005007720179624 -0.0029087196307811913"/>
+    <origin xyz="0.0 0.0 1.4500000000000002" rpy="0.0 -0.0 0.0"/>
     <parent link="base_link"/>
     <child link="top_laser_base_link"/>
@@ -234,5 +240,5 @@
   </link>
   <gazebo reference="top_laser">
-    <sensor name="top_laser-VLP16" type="gpu_ray">
+    <sensor name="top_laser-VLP16" type="ray">
       <pose>0 0 0 0 0 0</pose>
       <visualize>false</visualize>
@@ -264,5 +270,5 @@
         </noise>
       </ray>
-      <plugin filename="libgazebo_ros_velodyne_gpu_laser.so" name="gazebo_ros_laser_controller">
+      <plugin filename="libgazebo_ros_velodyne_laser.so" name="gazebo_ros_laser_controller">
         <topicName>top_laser/cloud</topicName>
         <frameName>top_laser</frameName>
@@ -642,3 +648,17 @@
     <material>Gazebo/Purple</material>
   </gazebo>
+  <link name="pattern_link">
+    <origin xyz="0 0 0" rpy="0 0 0"/>
+    <visual name="pattern_1_visual">
+      <origin xyz="0 0 0" rpy="0 0 0"/>
+      <geometry>
+        <mesh filename="package://atlascar2_gazebo/models/charuco_800x600/charuco_800x600.dae"/>
+      </geometry>
+    </visual>
+  </link>
+  <joint name="world-pattern_link" type="fixed">
+    <origin xyz="2.1196767724022947 0.11115631356790558 1.7810701835098057" rpy="-1.6196809177686766 0.9538883423404817 -1.6106085746501164"/>
+    <parent link="world"/>
+    <child link="pattern_link"/>
+  </joint>
 </robot>

File: atlascar2_description/urdf/atlascar2_ackermann_VLP.urdf.xacro (robot description, xacro)
@@ -24,4 +24,10 @@
     <xacro:atlascar2 length="${length}" width="${width}" height="${height}" wheel_radius="${wheel_radius}"/>
     <!--    Add sensors-->
+    <!-- <link name="world" />
+    <joint name="world_to_base_footprint" type="fixed">
+        <parent link="world" />
+        <child link="base_footprint" />
+        <origin xyz="0 0 0" rpy="0 0 0" />
+    </joint> -->
     <!-- top-right-camera -->
     <xacro:pointgrey_flea3_joints name="top_right_camera" frame="top_right_camera" parent="base_link"
