Commit message: .

File: atlascar2_calibration/urdf/initial_estimate.urdf.xacro (robot description, xacro)
@@ -1,92 +1,530 @@
-<?xml version="1.0"?>
-<robot name="atlascar2" xmlns:xacro="http://www.ros.org/wiki/xacro">
-    <!--
-    Robot model taken from http://wiki.ros.org/pr2_mechanism/Tutorials/SImple%20URDF-Controller%20Example
-    -->
-    <xacro:include filename="$(find atlascar2_description)/urdf/atlascar2_wheel.urdf.xacro"/>
-    <xacro:include filename="$(find atlascar2_description)/urdf/atlascar2_ackermann.macro.urdf.xacro"/>
-    <xacro:include filename="$(find velodyne_description)/urdf/VLP-16.urdf.xacro"/>
-    <!-- <xacro:include filename="$(find sick_ldmrs_description)/urdf/sick_ldmrs_macros.urdf.xacro"/> -->
-    <xacro:property name="deg_to_rad" value="0.01745329251994329577"/>
-    <!-- Constants for robot dimensions -->
-    <xacro:property name="length" value="3.475" />
-    <xacro:property name="width" value="1.475" />
-    <xacro:property name="height" value="1.61"/>
-    <xacro:property name="length_offset" value="0.2"/>
-    <xacro:property name="height_offset" value="0.1"/>
-    <xacro:property name="wheel_radius" value="0.285" /> <!-- Link 1 -->
-    <xacro:property name="thickness" value="0.145" /> <!-- Link 2 -->
-    <!--  we need two because the car isn't a square-->
-    <xacro:property name="axel_offset_x" value="0.5" /> <!-- Space btw top of beam and the each joint -->
-    <xacro:property name="axel_offset_y" value="0" /> <!-- Space btw top of beam and the each joint -->
-    <xacro:property name="steer_offset" value="0.02" /> <!-- Link 1 -->
-    <!-- Add car macro -->
-    <xacro:atlascar2 length="${length}" width="${width}" height="${height}" wheel_radius="${wheel_radius}"/>
-    <!--    Add sensors-->
-    <!-- <link name="world" />
-    <joint name="world_to_base_footprint" type="fixed">
-        <parent link="world" />
-        <child link="base_footprint" />
-        <origin xyz="0 0 0" rpy="0 0 0" />
-    </joint> -->
-    <!-- top-right-camera -->
-    <xacro:pointgrey_flea3_joints name="top_right_camera" frame="top_right_camera" parent="base_link"
-                                  x="${length_offset}" y="-0.22" z="${1.35+height_offset}"
-                                  rol="0" pit="0.4" yaw="0"/>
-    <!-- top-left-camera -->
-    <xacro:pointgrey_flea3_joints name="top_left_camera" frame="top_left_camera" parent="base_link"
-                                  x="${length_offset}" y="0.22" z="${1.35+height_offset}"
-                                  rol="0" pit="0.4" yaw="0"/>
-    <!-- top velodyne lidar -->
-    <xacro:VLP-16 name="top_laser" parent="base_link" topic="top_laser/cloud">
-      <origin xyz="0 0 ${1.35+height_offset}" rpy="0 0 0"/>
-    </xacro:VLP-16>
-    <!-- joints for ackermann_steering_controller -->
-    <xacro:front_steer name="front" parent="base" radius="${wheel_radius}" thickness="${thickness}"
-                       length="${length}" width="${width}" axel_offset="${axel_offset_x}" steer_height="${wheel_radius+steer_offset}">
-        <origin xyz="${length/2-axel_offset_x} 0 0" rpy="${-90 * deg_to_rad} 0 ${90 * deg_to_rad}"/>
-    </xacro:front_steer>
-    <xacro:rear_wheel name="rear" parent="base" radius="${wheel_radius}" thickness="${thickness}">
-        <origin xyz="${-length/2+axel_offset_x} 0 0" rpy="${-90 * deg_to_rad} 0 ${-90 * deg_to_rad}"/>
-    </xacro:rear_wheel>
-    <!-- laser sensor lms_ldmrs400001 -->
-    <!-- <xacro:sick_ldmrs name="frontal_laser"/> -->
-    <!-- <joint name="base_link_to_frontal_laser_mount_link" type="fixed"> -->
-      <!-- <origin xyz="${length/2 + length_offset} 0 ${height_offset}" rpy="0 0 0"/> -->
-      <!-- <parent link="base_link"/> -->
-      <!-- <child link="frontal_laser_mount_link"/> -->
-    <!-- </joint> -->
-    <!-- left lms151 laser -->
-    <xacro:sick_lms1xx_joints frame="left_laser" topic="/left_laser/scan" parent="base_link"
-                                  x="${length/2 + length_offset - 0.08}" y="0.76" z="${0.27+height_offset}"
-                                  rol="0" pit="0" yaw="0.7854"/>
-    <!-- right lms151 laser -->
-    <xacro:sick_lms1xx_joints frame="right_laser" topic="/right_laser/scan" parent="base_link"
-                                  x="${length/2 + length_offset - 0.08}" y="-0.76" z="${0.27+height_offset}"
-                                  rol="0" pit="0" yaw="-0.7854"/>
-    <!-- Wheels -->
-    <xacro:front_wheel_lr name="front_right" parent="base" radius="${wheel_radius}" thickness="${thickness}"
-                          length="${length}" width="${width}" axel_offset="${axel_offset_x}" right_left="1" steer_height="${wheel_radius+steer_offset}">
-        <origin xyz="${length/2-axel_offset_x} ${width/2+axel_offset_y} 0" rpy="${-90 * deg_to_rad} 0 0"/>
-    </xacro:front_wheel_lr>
-    <xacro:front_wheel_lr name="front_left" parent="base" radius="${wheel_radius}" thickness="${thickness}"
-                          length="${length}" width="${width}" axel_offset="${axel_offset_x}" right_left="-1" steer_height="${wheel_radius+steer_offset}">
-        <origin xyz="${length/2-axel_offset_x} ${-width/2-axel_offset_y} 0" rpy="${-90 * deg_to_rad} 0 0"/>
-    </xacro:front_wheel_lr>
-    <xacro:rear_wheel_lr name="rear_right" parent="base" radius="${wheel_radius}" right_left="1" thickness="${thickness}">
-        <origin xyz="${-length/2+axel_offset_x - 0.05} ${width/2+axel_offset_y} 0" rpy="${-90 * deg_to_rad} 0 ${-90 * deg_to_rad}"/>
-    </xacro:rear_wheel_lr>
-    <xacro:rear_wheel_lr name="rear_left" parent="base" radius="${wheel_radius}" right_left="-1" thickness="${thickness}">
-        <origin xyz="${-length/2+axel_offset_x - 0.05} ${-width/2-axel_offset_y} 0" rpy="${-90 * deg_to_rad} 0 ${90 * deg_to_rad}"/>
-    </xacro:rear_wheel_lr>
-    <!-- Gazebo plugin for ROS Control -->
-    <gazebo>
-        <plugin name="gazebo_ros_control" filename="libgazebo_ros_control.so">
-            <robotSimType>steer_bot_hardware_gazebo/SteerBotHardwareGazebo</robotSimType>
-        </plugin>
-    </gazebo>
-    <!-- Colour -->
-    <gazebo reference="base_footprint">
-        <material>Gazebo/Purple</material>
-    </gazebo>
+<?xml version="1.0" ?>
+<robot name="atlascar2" version="1.0">
+  <link name="base_link">
+    <inertial>
+      <origin xyz="0.0 0.0 0.0" rpy="0.0 0.0 0.0"/>
+      <mass value="2.0"/>
+      <inertia ixx="1.0" ixy="0.0" ixz="0.0" iyy="1.0" iyz="0.0" izz="1.0"/>
+    </inertial>
+    <visual>
+      <origin xyz="1.7375 -0.8875000000000001 -0.235" rpy="0.0 0.0 1.5707963267948966"/>
+      <geometry>
+        <mesh filename="file:////home/rafael/catkin_ws/src/atlascar2/atlascar2_description/meshes/atlascar2_nowheels.dae"/>
+      </geometry>
+    </visual>
+    <collision>
+      <origin xyz="0.0 0.0 0.52" rpy="0 0 0"/>
+      <geometry>
+        <box size="3.375 1.475 0.805"/>
+      </geometry>
+    </collision>
+  </link>
+  <link name="top_collision">
+    <collision>
+      <origin xyz="-0.49642857142857144 0.0 0.0" rpy="0 0 0"/>
+      <geometry>
+        <box size="1.7375 1.475 0.805"/>
+      </geometry>
+    </collision>
+  </link>
+  <joint name="base_link_to_top_collision" type="fixed">
+    <origin xyz="0.0 0.0 0.805" rpy="0.0 0.0 0.0"/>
+    <parent link="base_link"/>
+    <child link="top_collision"/>
+  </joint>
+  <link name="base_footprint">
+    <collision>
+      <origin xyz="0.0 0.0 0.0" rpy="0 0 0"/>
+      <geometry>
+        <sphere radius="1e-08"/>
+      </geometry>
+    </collision>
+  </link>
+  <joint name="base_footprint_joint" type="fixed">
+    <origin xyz="0.0 0.0 0.285" rpy="0.0 0.0 0.0"/>
+    <parent link="base_footprint"/>
+    <child link="base_link"/>
+  </joint>
+  <link name="top_left_camera">
+    <inertial>
+      <mass value="0.085"/>
+      <inertia ixx="1e-06" ixy="0.0" ixz="0.0" iyy="1e-06" iyz="0.0" izz="1e-06"/>
+    </inertial>
+    <visual>
+      <origin xyz="0.0 0.0 0.0" rpy="0.0 0.0 0.0"/>
+      <geometry>
+        <box size="0.0754 0.029 0.035"/>
+      </geometry>
+      <material name="dark_grey"/>
+    </visual>
+    <collision>
+      <origin xyz="0.0 0.0 0.0" rpy="0.0 0.0 0.0"/>
+      <geometry>
+        <box size="0.0754 0.029 0.035"/>
+      </geometry>
+    </collision>
+  </link>
+  <link name="top_left_camera_optical"/>
+  <joint name="top_left_camera_optical_joint" type="fixed">
+    <origin xyz="0.0 0.0 0.0" rpy="-1.570796 0.0 -1.570796"/>
+    <parent link="top_left_camera"/>
+    <child link="top_left_camera_optical"/>
+  </joint>
+  <gazebo reference="top_left_camera_optical">
+    <material>Gazebo/Grey</material>
+    <sensor name="top_left_camera" type="camera">
+      <update_rate>120</update_rate>
+      <camera name="top_left_camera">
+        <pose>0 0 0 0 -1.5707 1.5707</pose>
+        <horizontal_fov>1.0471975512</horizontal_fov>
+        <image>
+          <width>1272</width>
+          <height>1016</height>
+          <format>R8G8B8</format>
+        </image>
+        <clip>
+          <near>0.5</near>
+          <far>300</far>
+        </clip>
+        <noise>
+          <type>gaussian</type>
+          <mean>0.0</mean>
+          <stddev>0.007</stddev>
+        </noise>
+      </camera>
+      <plugin filename="libgazebo_ros_camera.so" name="camera_controller">
+        <alwaysOn>true</alwaysOn>
+        <updateRate>120</updateRate>
+        <cameraName>top_left_camera</cameraName>
+        <imageTopicName>image_raw</imageTopicName>
+        <cameraInfoTopicName>camera_info</cameraInfoTopicName>
+        <frameName>top_left_camera_optical</frameName>
+        <hackBaseline>0.07</hackBaseline>
+        <distortionK1>0.0</distortionK1>
+        <distortionK2>0.0</distortionK2>
+        <distortionK3>0.0</distortionK3>
+        <distortionT1>0.0</distortionT1>
+        <distortionT2>0.0</distortionT2>
+      </plugin>
+    </sensor>
+  </gazebo>
+  <joint name="{parent}_to_top_left_camera" type="fixed">
+    <origin xyz="0.6000000238418579 0.3499999940395355 1.2949999570846558" rpy="-0.0020112537709440683 -0.00471036429682682 0.40356578749296457"/>
+    <parent link="base_link"/>
+    <child link="top_left_camera"/>
+  </joint>
+  <joint name="top_right_camera_joint" type="fixed">
+    <origin xyz="0.5 -0.27000001072883606 1.3450000286102295" rpy="0.0050055992379940345 -0.03278777944374682 -0.15152288325436902"/>
+    <parent link="base_link"/>
+    <child link="top_right_camera"/>
+  </joint>
+  <link name="top_right_camera">
+    <inertial>
+      <origin xyz="0.0 0.0 0.0" rpy="0 0 0"/>
+      <mass value="0.00564"/>
+      <inertia ixx="0.003881243" ixy="0.0" ixz="0.0" iyy="0.00049894" iyz="0.0" izz="0.003879257"/>
+    </inertial>
+    <visual>
+      <origin xyz="0.0 0.0 0.0" rpy="0.0 0.0 0.0"/>
+      <geometry>
+        <mesh filename="package://atlascar2_description/meshes/rgb_camera/rgb_camera.stl" scale="1.0 1.0 1.0"/>
+      </geometry>
+      <material name="green">
+        <color rgba="0.0 0.9 0.0 1.0"/>
+      </material>
+    </visual>
+    <collision>
+      <origin xyz="0.0 0.0 0.0" rpy="0.0 0.0 0.0"/>
+      <geometry>
+        <mesh filename="package://atlascar2_description/meshes/rgb_camera/rgb_camera.stl" scale="1.0 1.0 1.0"/>
+      </geometry>
+    </collision>
+  </link>
+  <gazebo reference="top_right_camera">
+    <selfCollide>false</selfCollide>
+    <material>Gazebo/Green</material>
+  </gazebo>
+  <joint name="top_right_camera_optical_joint" type="fixed">
+    <origin xyz="0.0 0.0 0.0" rpy="-1.5707963267948966 0.0 -1.5707963267948966"/>
+    <parent link="top_right_camera"/>
+    <child link="top_right_camera_optical"/>
+  </joint>
+  <link name="top_right_camera_optical"/>
+  <gazebo reference="top_right_camera_link">
+    <sensor name="camera" type="camera">
+      <update_rate>10.0</update_rate>
+      <camera>
+        <horizontal_fov>1.0471975511965976</horizontal_fov>
+        <image>
+          <format>B8G8R8</format>
+          <width>1200</width>
+          <height>800</height>
+        </image>
+        <clip>
+          <near>0.10</near>
+          <far>8.0</far>
+        </clip>
+      </camera>
+      <plugin filename="libgazebo_ros_camera.so" name="top_right_camera_rgb_camera_controller">
+        <cameraName>top_right_camera</cameraName>
+        <alwaysOn>true</alwaysOn>
+        <updateRate>0</updateRate>
+        <imageTopicName>image_raw</imageTopicName>
+        <cameraInfoTopicName>camera_info</cameraInfoTopicName>
+        <frameName>top_right_camera_optical_frame</frameName>
+        <baseline>0.0</baseline>
+        <distortion_k1>0.0</distortion_k1>
+        <distortion_k2>0.0</distortion_k2>
+        <distortion_k3>0.0</distortion_k3>
+        <distortion_t1>0.0</distortion_t1>
+        <distortion_t2>0.0</distortion_t2>
+      </plugin>
+    </sensor>
+  </gazebo>
+  <joint name="top_laser_base_mount_joint" type="fixed">
+    <origin xyz="0.5 0.0 1.515" rpy="0.0 -0.0 0.0"/>
+    <parent link="base_link"/>
+    <child link="top_laser_base_link"/>
+  </joint>
+  <link name="top_laser_base_link">
+    <inertial>
+      <origin xyz="0.0 0.0 0.03585" rpy="0 0 0"/>
+      <mass value="0.83"/>
+      <inertia ixx="0.000908059425" ixy="0.0" ixz="0.0" iyy="0.000908059425" iyz="0.0" izz="0.0011049624"/>
+    </inertial>
+    <visual>
+      <geometry>
+        <mesh filename="package://velodyne_description/meshes/VLP16_base_1.dae"/>
+      </geometry>
+    </visual>
+    <visual>
+      <geometry>
+        <mesh filename="package://velodyne_description/meshes/VLP16_base_2.dae"/>
+      </geometry>
+    </visual>
+    <collision>
+      <origin xyz="0.0 0.0 0.03585" rpy="0.0 0.0 0.0"/>
+      <geometry>
+        <cylinder radius="0.0516" length="0.0717"/>
+      </geometry>
+    </collision>
+  </link>
+  <joint name="top_laser_base_scan_joint" type="fixed">
+    <origin xyz="0.0 0.0 0.0377" rpy="0.0 0.0 0.0"/>
+    <parent link="top_laser_base_link"/>
+    <child link="top_laser"/>
+  </joint>
+  <link name="top_laser">
+    <inertial>
+      <origin xyz="0.0 0.0 0.0" rpy="0 0 0"/>
+      <mass value="0.01"/>
+      <inertia ixx="1e-07" ixy="0.0" ixz="0.0" iyy="1e-07" iyz="0.0" izz="1e-07"/>
+    </inertial>
+    <visual>
+      <origin xyz="0.0 0.0 -0.0377" rpy="0 0 0"/>
+      <geometry>
+        <mesh filename="package://velodyne_description/meshes/VLP16_scan.dae"/>
+      </geometry>
+    </visual>
+    <collision>
+      <geometry>
+        <sphere radius="0.0"/>
+      </geometry>
+    </collision>
+  </link>
+  <gazebo reference="top_laser">
+    <sensor name="top_laser-VLP16" type="ray">
+      <pose>0 0 0 0 0 0</pose>
+      <visualize>false</visualize>
+      <update_rate>10</update_rate>
+      <ray>
+        <scan>
+          <horizontal>
+            <samples>1875</samples>
+            <resolution>1</resolution>
+            <min_angle>-3.141592653589793</min_angle>
+            <max_angle>3.141592653589793</max_angle>
+          </horizontal>
+          <vertical>
+            <samples>16</samples>
+            <resolution>1</resolution>
+            <min_angle>-0.2617993877991494</min_angle>
+            <max_angle> 0.2617993877991494</max_angle>
+          </vertical>
+        </scan>
+        <range>
+          <min>0.3</min>
+          <max>131.0</max>
+          <resolution>0.001</resolution>
+        </range>
+        <noise>
+          <type>gaussian</type>
+          <mean>0.0</mean>
+          <stddev>0.0</stddev>
+        </noise>
+      </ray>
+      <plugin filename="libgazebo_ros_velodyne_laser.so" name="gazebo_ros_laser_controller">
+        <topicName>/top_laser/cloud</topicName>
+        <frameName>top_laser</frameName>
+        <organize_cloud>False</organize_cloud>
+        <min_range>0.9</min_range>
+        <max_range>130.0</max_range>
+        <gaussianNoise>0.008</gaussianNoise>
+      </plugin>
+    </sensor>
+  </gazebo>
+  <link name="front_steer_link">
+    <inertial>
+      <origin xyz="0.0 0.0 0.0" rpy="0.0 0.0 0.0"/>
+      <mass value="11.16"/>
+      <inertia ixx="0.246171" ixy="0.0" ixz="0.0" iyy="0.246171" iyz="0.0" izz="0.4532354999999999"/>
+    </inertial>
+    <collision>
+      <origin xyz="0.0 0.0 0.0" rpy="0.0 0.0 0.0"/>
+      <geometry>
+        <cylinder radius="0.05" length="0.02"/>
+      </geometry>
+    </collision>
+  </link>
+  <joint name="front_steer_joint" type="revolute">
+    <origin xyz="1.2375 0.0 0.305" rpy="0.0 0.0 0.0"/>
+    <axis xyz="0.0 0.0 1.0"/>
+    <parent link="base_link"/>
+    <child link="front_steer_link"/>
+    <limit effort="15.0" lower="-3.141592653589793" upper="3.141592653589793" velocity="5.0"/>
+    <dynamics damping="0.0" friction="0.0"/>
+  </joint>
+  <transmission name="front_steer_joint_trans">
+    <type>transmission_interface/SimpleTransmission</type>
+    <actuator name="front_steer_joint_motor"/>
+    <joint name="front_steer_joint">
+      <hardwareInterface>hardware_interface/PositionJointInterface</hardwareInterface>
+    </joint>
+  </transmission>
+  <gazebo reference="front_steer_link">
+    <material>Gazebo/Yellow</material>
+  </gazebo>
+  <link name="rear_wheel_link">
+    <inertial>
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