Commit message: .

File: atlascar2_calibration/urdf/optimized_simulation.urdf.xacro (robot description, xacro)
@@ -45,4 +45,72 @@
     <parent link="base_footprint"/>
     <child link="base_link"/>
+  </joint>
+  <link name="top_right_camera">
+    <inertial>
+      <mass value="0.085"/>
+      <inertia ixx="1e-06" ixy="0.0" ixz="0.0" iyy="1e-06" iyz="0.0" izz="1e-06"/>
+    </inertial>
+    <visual>
+      <origin xyz="0.0 0.0 0.0" rpy="0.0 0.0 0.0"/>
+      <geometry>
+        <box size="0.0754 0.029 0.035"/>
+      </geometry>
+      <material name="dark_grey"/>
+    </visual>
+    <collision>
+      <origin xyz="0.0 0.0 0.0" rpy="0.0 0.0 0.0"/>
+      <geometry>
+        <box size="0.0754 0.029 0.035"/>
+      </geometry>
+    </collision>
+  </link>
+  <link name="top_right_camera_optical"/>
+  <joint name="top_right_camera_optical_joint" type="fixed">
+    <origin xyz="0.0 0.0 0.0" rpy="-1.570796 0.0 -1.570796"/>
+    <parent link="top_right_camera"/>
+    <child link="top_right_camera_optical"/>
+  </joint>
+  <gazebo reference="top_right_camera_optical">
+    <material>Gazebo/Grey</material>
+    <sensor name="top_right_camera" type="camera">
+      <update_rate>120</update_rate>
+      <camera name="top_right_camera">
+        <pose>0 0 0 0 -1.5707 1.5707</pose>
+        <horizontal_fov>1.0471975512</horizontal_fov>
+        <image>
+          <width>1272</width>
+          <height>1016</height>
+          <format>R8G8B8</format>
+        </image>
+        <clip>
+          <near>0.5</near>
+          <far>300</far>
+        </clip>
+        <noise>
+          <type>gaussian</type>
+          <mean>0.0</mean>
+          <stddev>0.007</stddev>
+        </noise>
+      </camera>
+      <plugin filename="libgazebo_ros_camera.so" name="camera_controller">
+        <alwaysOn>true</alwaysOn>
+        <updateRate>120</updateRate>
+        <cameraName>top_right_camera</cameraName>
+        <imageTopicName>image_raw</imageTopicName>
+        <cameraInfoTopicName>camera_info</cameraInfoTopicName>
+        <frameName>top_right_camera_optical</frameName>
+        <hackBaseline>0.07</hackBaseline>
+        <distortionK1>0.0</distortionK1>
+        <distortionK2>0.0</distortionK2>
+        <distortionK3>0.0</distortionK3>
+        <distortionT1>0.0</distortionT1>
+        <distortionT2>0.0</distortionT2>
+      </plugin>
+    </sensor>
+  </gazebo>
+  <joint name="{parent}_to_top_right_camera" type="fixed">
+    <origin xyz="0.20428410540814848 -0.22388230247232627 1.447061150205553" rpy="-0.00042622049778580357 0.3 -0.3"/>
+    <parent link="base_link"/>
+    <child link="top_right_camera"/>
   </joint>
   <link name="top_left_camera">
@@ -110,78 +178,10 @@
   </gazebo>
   <joint name="{parent}_to_top_left_camera" type="fixed">
-    <origin xyz="0.6466467301243726 0.3406895632742394 1.294151091127127" rpy="-0.01626691548060342 -0.005101236526765667 0.4110508093626245"/>
+    <origin xyz="0.20000000000000043 0.22000000000000017 1.4500000000000002" rpy="-1.5554606490236454e-16 0.3 0.3"/>
     <parent link="base_link"/>
     <child link="top_left_camera"/>
   </joint>
-  <joint name="top_right_camera_joint" type="fixed">
-    <origin xyz="0.45708507829916045 -0.2668261665626715 1.345833073821856" rpy="-0.0026675009053780258 -0.029910542110388037 -0.15692317777900808"/>
-    <parent link="base_link"/>
-    <child link="top_right_camera"/>
-  </joint>
-  <link name="top_right_camera">
-    <inertial>
-      <origin xyz="0.0 0.0 0.0" rpy="0 0 0"/>
-      <mass value="0.00564"/>
-      <inertia ixx="0.003881243" ixy="0.0" ixz="0.0" iyy="0.00049894" iyz="0.0" izz="0.003879257"/>
-    </inertial>
-    <visual>
-      <origin xyz="0.0 0.0 0.0" rpy="0.0 0.0 0.0"/>
-      <geometry>
-        <mesh filename="package://atlascar2_description/meshes/rgb_camera/rgb_camera.stl" scale="1.0 1.0 1.0"/>
-      </geometry>
-      <material name="green">
-        <color rgba="0.0 0.9 0.0 1.0"/>
-      </material>
-    </visual>
-    <collision>
-      <origin xyz="0.0 0.0 0.0" rpy="0.0 0.0 0.0"/>
-      <geometry>
-        <mesh filename="package://atlascar2_description/meshes/rgb_camera/rgb_camera.stl" scale="1.0 1.0 1.0"/>
-      </geometry>
-    </collision>
-  </link>
-  <gazebo reference="top_right_camera">
-    <selfCollide>false</selfCollide>
-    <material>Gazebo/Green</material>
-  </gazebo>
-  <joint name="top_right_camera_optical_joint" type="fixed">
-    <origin xyz="0.0 0.0 0.0" rpy="-1.5707963267948966 0.0 -1.5707963267948966"/>
-    <parent link="top_right_camera"/>
-    <child link="top_right_camera_optical"/>
-  </joint>
-  <link name="top_right_camera_optical"/>
-  <gazebo reference="top_right_camera_link">
-    <sensor name="camera" type="camera">
-      <update_rate>10.0</update_rate>
-      <camera>
-        <horizontal_fov>1.0471975511965976</horizontal_fov>
-        <image>
-          <format>B8G8R8</format>
-          <width>1200</width>
-          <height>800</height>
-        </image>
-        <clip>
-          <near>0.10</near>
-          <far>8.0</far>
-        </clip>
-      </camera>
-      <plugin filename="libgazebo_ros_camera.so" name="top_right_camera_rgb_camera_controller">
-        <cameraName>top_right_camera</cameraName>
-        <alwaysOn>true</alwaysOn>
-        <updateRate>0</updateRate>
-        <imageTopicName>image_raw</imageTopicName>
-        <cameraInfoTopicName>camera_info</cameraInfoTopicName>
-        <frameName>top_right_camera_optical_frame</frameName>
-        <baseline>0.0</baseline>
-        <distortion_k1>0.0</distortion_k1>
-        <distortion_k2>0.0</distortion_k2>
-        <distortion_k3>0.0</distortion_k3>
-        <distortion_t1>0.0</distortion_t1>
-        <distortion_t2>0.0</distortion_t2>
-      </plugin>
-    </sensor>
-  </gazebo>
   <joint name="top_laser_base_mount_joint" type="fixed">
-    <origin xyz="0.5105322445361739 -0.04054793927958642 1.4740715062770289" rpy="-0.010912443904387446 -0.012832418570686559 0.017753230379700616"/>
+    <origin xyz="0.016363087328487538 0.01008967362563249 1.4746227815305066" rpy="-0.0022630437000740813 0.010005007720179624 -0.0029087196307811913"/>
     <parent link="base_link"/>
     <child link="top_laser_base_link"/>
@@ -234,5 +234,5 @@
   </link>
   <gazebo reference="top_laser">
-    <sensor name="top_laser-VLP16" type="ray">
+    <sensor name="top_laser-VLP16" type="gpu_ray">
       <pose>0 0 0 0 0 0</pose>
       <visualize>false</visualize>
@@ -264,6 +264,6 @@
         </noise>
       </ray>
-      <plugin filename="libgazebo_ros_velodyne_laser.so" name="gazebo_ros_laser_controller">
-        <topicName>/top_laser/cloud</topicName>
+      <plugin filename="libgazebo_ros_velodyne_gpu_laser.so" name="gazebo_ros_laser_controller">
+        <topicName>top_laser/cloud</topicName>
         <frameName>top_laser</frameName>
         <organize_cloud>False</organize_cloud>
@@ -332,4 +332,118 @@
     </joint>
   </transmission>
+  <link name="left_laser">
+    <inertial>
+      <origin xyz="0.0 0.0 0.0" rpy="0 0 0"/>
+      <mass value="1.1"/>
+      <inertia ixx="0.00307156543804" ixy="0.0" ixz="0.0" iyy="0.0031284904152700005" iyz="0.0" izz="0.00196432421427"/>
+    </inertial>
+    <visual>
+      <origin xyz="0.0 0.0 0.0" rpy="0.0 0.0 0.0"/>
+      <geometry>
+        <mesh filename="package://lms1xx/meshes/sick-lms1xx.dae"/>
+      </geometry>
+    </visual>
+    <collision>
+      <origin xyz="0.0 0.0 -0.05" rpy="0.0 0.0 0.0"/>
+      <geometry>
+        <box size="0.105 0.1 0.1"/>
+      </geometry>
+    </collision>
+  </link>
+  <gazebo reference="left_laser">
+    <turnGravityOff>true</turnGravityOff>
+    <sensor name="left_laser" type="ray">
+      <pose>0 0 0 0 0 0</pose>
+      <visualize>false</visualize>
+      <update_rate>50</update_rate>
+      <ray>
+        <scan>
+          <horizontal>
+            <samples>720</samples>
+            <resolution>1</resolution>
+            <min_angle>-2.35619</min_angle>
+            <max_angle>2.35619</max_angle>
+          </horizontal>
+        </scan>
+        <range>
+          <min>0.1</min>
+          <max>30.0</max>
+          <resolution>0.01</resolution>
+        </range>
+        <noise>
+          <type>gaussian</type>
+          <mean>0.0</mean>
+          <stddev>0.001</stddev>
+        </noise>
+      </ray>
+      <plugin filename="libgazebo_ros_laser.so" name="gazebo_ros_laser">
+        <topicName>/left_laser/scan</topicName>
+        <frameName>left_laser</frameName>
+        <robotNamespace>/</robotNamespace>
+      </plugin>
+    </sensor>
+  </gazebo>
+  <joint name="{parent}_to_left_laser" type="fixed">
+    <origin xyz="1.8575 0.76 0.37" rpy="0.0 0.0 0.7854"/>
+    <parent link="base_link"/>
+    <child link="left_laser"/>
+  </joint>
+  <link name="right_laser">
+    <inertial>
+      <origin xyz="0.0 0.0 0.0" rpy="0 0 0"/>
+      <mass value="1.1"/>
+      <inertia ixx="0.00307156543804" ixy="0.0" ixz="0.0" iyy="0.0031284904152700005" iyz="0.0" izz="0.00196432421427"/>
+    </inertial>
+    <visual>
+      <origin xyz="0.0 0.0 0.0" rpy="0.0 0.0 0.0"/>
+      <geometry>
+        <mesh filename="package://lms1xx/meshes/sick-lms1xx.dae"/>
+      </geometry>
+    </visual>
+    <collision>
+      <origin xyz="0.0 0.0 -0.05" rpy="0.0 0.0 0.0"/>
+      <geometry>
+        <box size="0.105 0.1 0.1"/>
+      </geometry>
+    </collision>
+  </link>
+  <gazebo reference="right_laser">
+    <turnGravityOff>true</turnGravityOff>
+    <sensor name="right_laser" type="ray">
+      <pose>0 0 0 0 0 0</pose>
+      <visualize>false</visualize>
+      <update_rate>50</update_rate>
+      <ray>
+        <scan>
+          <horizontal>
+            <samples>720</samples>
+            <resolution>1</resolution>
+            <min_angle>-2.35619</min_angle>
+            <max_angle>2.35619</max_angle>
+          </horizontal>
+        </scan>
+        <range>
+          <min>0.1</min>
+          <max>30.0</max>
+          <resolution>0.01</resolution>
+        </range>
+        <noise>
+          <type>gaussian</type>
+          <mean>0.0</mean>
+          <stddev>0.001</stddev>
+        </noise>
+      </ray>
+      <plugin filename="libgazebo_ros_laser.so" name="gazebo_ros_laser">
+        <topicName>/right_laser/scan</topicName>
+        <frameName>right_laser</frameName>
+        <robotNamespace>/</robotNamespace>
+      </plugin>
+    </sensor>
+  </gazebo>
+  <joint name="{parent}_to_right_laser" type="fixed">
+    <origin xyz="1.8575 -0.76 0.37" rpy="0.0 0.0 -0.7854"/>
+    <parent link="base_link"/>
+    <child link="right_laser"/>
+  </joint>
   <link name="front_right_steer_link">
     <inertial>
