Commit message: .

File: atlascar2_calibration/urdf/optimized.urdf.xacro (robot description, xacro)
@@ -110,5 +110,5 @@
   </gazebo>
   <joint name="{parent}_to_top_right_camera" type="fixed">
-    <origin xyz="0.20428410540814848 -0.22388230247232627 1.447061150205553" rpy="-0.00042622049778580357 0.3988143668006885 -0.3"/>
+    <origin xyz="0.20428410540814848 -0.22388230247232627 1.447061150205553" rpy="-0.00042622049778580357 0.3 -0.3"/>
     <parent link="base_link"/>
     <child link="top_right_camera"/>
@@ -178,5 +178,5 @@
   </gazebo>
   <joint name="{parent}_to_top_left_camera" type="fixed">
-    <origin xyz="0.20000000000000043 0.22000000000000017 1.4500000000000002" rpy="-1.5554606490236454e-16 0.4 0.3"/>
+    <origin xyz="0.20000000000000043 0.22000000000000017 1.4500000000000002" rpy="-1.5554606490236454e-16 0.3 0.3"/>
     <parent link="base_link"/>
     <child link="top_left_camera"/>

Commit message: .

File: atlascar2_calibration/urdf/optimized.urdf.xacro (robot description, xacro)
@@ -110,5 +110,5 @@
   </gazebo>
   <joint name="{parent}_to_top_left_camera" type="fixed">
-    <origin xyz="0.6466467301243726 0.3406895632742394 1.294151091127127" rpy="-0.01626691548060342 -0.005101236526765667 0.4110508093626245"/>
+    <origin xyz="0.6466467301243726 0.3406895632742394 1.294151091127127" rpy="-0.01626691548060342 -0.005101236526765667 0.45110508093626245"/>
     <parent link="base_link"/>
     <child link="top_left_camera"/>

Commit message: Revert "."
This reverts commit c2a3c3f39755477d3054d07457dcc350ad674e3a.

File: atlascar2_calibration/urdf/optimized.urdf.xacro (robot description, xacro)
@@ -110,5 +110,5 @@
   </gazebo>
   <joint name="{parent}_to_top_left_camera" type="fixed">
-    <origin xyz="0.6466467301243726 0.3406895632742394 1.294151091127127" rpy="-0.01626691548060342 -0.005101236526765667 0.45110508093626245"/>
+    <origin xyz="0.6466467301243726 0.3406895632742394 1.294151091127127" rpy="-0.01626691548060342 -0.005101236526765667 0.4110508093626245"/>
     <parent link="base_link"/>
     <child link="top_left_camera"/>
